File: hardware/card/card.kicad_pcb (KiCad board)
At the start: 4 copper layers, 116 x 106 mm, 0 parts

Commit message: hardware: reset card PCB layout path
Changed lines of the file:
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@@
   (gr_text "SW_RESTART" (at 92 9.5 0) (layer "F.SilkS")
     (effects (font (size 1 1) (thickness 0.15)) (justify center)))
-  (gr_circle (center 30.5 4) (end 31 4) (stroke (width 0.12) (type default)) (fill none) (layer "F.Fab"))
-  (gr_text "SW_MENU" (at 30.5 5.5 0) (layer "F.SilkS")
+  (gr_circle (center 58 9) (end 58.5 9) (stroke (width 0.12) (type default)) (fill none) (layer "F.Fab"))
+  (gr_text "SW_MENU" (at 58 10.5 0) (layer "F.SilkS")
     (effects (font (size 1 1) (thickness 0.15)) (justify center)))
   (gr_circle (center 60 106.5) (end 60.5 106.5) (stroke (width 0.12) (type default)) (fill none) (layer "F.Fab"))
@@
   (gr_text "ACT_LRA" (at 100 20.5 0) (layer "F.SilkS")
     (effects (font (size 1 1) (thickness 0.15)) (justify center)))
-  (gr_circle (center 53 11) (end 53.5 11) (stroke (width 0.12) (type default)) (fill none) (layer "F.Fab"))
-  (gr_text "PAD_PIEZO" (at 53 12.5 0) (layer "F.SilkS")
+  (gr_circle (center 60 24) (end 60.5 24) (stroke (width 0.12) (type default)) (fill none) (layer "F.Fab"))
+  (gr_text "PAD_PIEZO" (at 60 25.5 0) (layer "F.SilkS")
     (effects (font (size 1 1) (thickness 0.15)) (justify center)))
   (gr_rect (start 7.29 39.43000000000001) (end 112.71000000000001 106.5) (stroke (width 0.12) (type dash)) (fill none) (layer "Eco1.User"))
-  (gr_rect (start 37 7) (end 69 37) (stroke (width 0.12) (type dash)) (fill none) (layer "Eco1.User"))
   (gr_rect (start 47 38) (end 73 110) (stroke (width 0.12) (type dash)) (fill none) (layer "Eco1.User"))
 )

Commit message: pcb stuff
Other:
- board text added: "action_support"
- board text added: "back_bat_1s_pouch"
- board text added: "back_esp32_p4_module"
- board text added: "back_pmic_cluster"
- board text added: "control_band"
- board text added: "display_active"
- board text added: "display_module"
- board text added: "dpad_support"
- board text added: "fpc_top_keepout"
Changed lines of the file:
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@@
   (gr_text "CONN_USB_C_MID" (at 25 109.5 0) (layer "F.SilkS")
     (effects (font (size 1 1) (thickness 0.15)) (justify center)))
-  (gr_circle (center 113 106.5) (end 113.5 106.5) (stroke (width 0.12) (type default)) (fill none) (layer "F.Fab"))
-  (gr_text "SW_POWER" (at 113 108 0) (layer "F.SilkS")
+  (gr_circle (center 106 106.5) (end 106.5 106.5) (stroke (width 0.12) (type default)) (fill none) (layer "F.Fab"))
+  (gr_text "SW_POWER" (at 106 108 0) (layer "F.SilkS")
     (effects (font (size 1 1) (thickness 0.15)) (justify center)))
   (gr_circle (center 118.5 92) (end 119 92) (stroke (width 0.12) (type default)) (fill none) (layer "F.Fab"))
@@
     (effects (font (size 1 1) (thickness 0.15)) (justify center)))
   (gr_rect (start 7.29 39.43000000000001) (end 112.71000000000001 106.5) (stroke (width 0.12) (type dash)) (fill none) (layer "Eco1.User"))
+  (gr_text "display_module" (at 60 108 0) (layer "Eco1.User")
+    (effects (font (size 1 1) (thickness 0.12)) (justify center)))
+  (gr_rect (start 12.5 46) (end 107.5 100) (stroke (width 0.12) (type dash)) (fill none) (layer "Cmts.User"))
+  (gr_text "display_active" (at 60 101.5 0) (layer "Cmts.User")
+    (effects (font (size 1 1) (thickness 0.12)) (justify center)))
   (gr_rect (start 47 38) (end 73 110) (stroke (width 0.12) (type dash)) (fill none) (layer "Eco1.User"))
+  (gr_text "fpc_top_keepout" (at 60 111.5 0) (layer "Eco1.User")
+    (effects (font (size 1 1) (thickness 0.12)) (justify center)))
+  (gr_rect (start 0 5) (end 120 38) (stroke (width 0.12) (type dash)) (fill none) (layer "Cmts.User"))
+  (gr_text "control_band" (at 60 39.5 0) (layer "Cmts.User")
+    (effects (font (size 1 1) (thickness 0.12)) (justify center)))
+  (gr_rect (start 8 9) (end 36 37) (stroke (width 0.12) (type dash)) (fill none) (layer "Dwgs.User"))
+  (gr_text "dpad_support" (at 22 38.5 0) (layer "Dwgs.User")
+    (effects (font (size 1 1) (thickness 0.12)) (justify center)))
+  (gr_rect (start 70 3) (end 100 33) (stroke (width 0.12) (type dash)) (fill none) (layer "Dwgs.User"))
+  (gr_text "action_support" (at 85 34.5 0) (layer "Dwgs.User")
+    (effects (font (size 1 1) (thickness 0.12)) (justify center)))
+  (gr_rect (start 31 7) (end 89 37) (stroke (width 0.12) (type dash)) (fill none) (layer "Eco2.User"))
+  (gr_text "back_bat_1s_pouch" (at 60 38.5 0) (layer "Eco2.User")
+    (effects (font (size 1 1) (thickness 0.12)) (justify center)))
+  (gr_rect (start 47.5 42) (end 72.5 67) (stroke (width 0.12) (type dash)) (fill none) (layer "Eco2.User"))
+  (gr_text "back_esp32_p4_module" (at 60 68.5 0) (layer "Eco2.User")
+    (effects (font (size 1 1) (thickness 0.12)) (justify center)))
+  (gr_rect (start 76 42) (end 98 53) (stroke (width 0.12) (type dash)) (fill none) (layer "Eco2.User"))
+  (gr_text "back_pmic_cluster" (at 87 54.5 0) (layer "Eco2.User")
+    (effects (font (size 1 1) (thickness 0.12)) (justify center)))
 )
