File: hardware/card/schematic/sheets/audio.kicad_sch (KiCad schematic)
At the start: 2 parts, among them Q1 NPN

Commit message: pcb stuff
Parts:
- added R7: 0R, 0402, symbol Device:R
- added U8: PiezoHBridge-DNP, TBD, symbol PSCard:Block2
Changed lines of the file:
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@@
     (instances (project "card" (path "/card/sheets/audio" (reference "JP1") (unit 1))))
   )
-  (label "GND" (at 98 32.5 0) (fields_autoplaced)
-    (effects (font (size 1.27 1.27)) (justify left)))
   (label "PIEZO_OUT" (at 98 30 0) (fields_autoplaced)
     (effects (font (size 1.27 1.27)) (justify left)))
-  (global_label "GND" (shape input) (at 280 20 0) (fields_autoplaced)
+  (label "PIEZO_RET" (at 98 32.5 0) (fields_autoplaced)
+    (effects (font (size 1.27 1.27)) (justify left)))
+  (symbol (lib_id "PSCard:Block2") (at 125 35 0) (unit 1)
+    (exclude_from_sim no) (in_bom yes) (on_board yes) (dnp no) (fields_autoplaced)
+    (property "Reference" "U8" (at 125 29 0)
+      (effects (font (size 1.27 1.27))))
+    (property "Value" "PiezoHBridge-DNP" (at 125 41 0)
+      (effects (font (size 1.27 1.27))))
+    (property "Footprint" "TBD" (at 125 35 0)
+      (effects (font (size 1.27 1.27)) hide))
+    (property "Datasheet" "~" (at 125 35 0)
+      (effects (font (size 1.27 1.27)) hide))
+    (instances (project "card" (path "/card/sheets/audio" (reference "U8") (unit 1))))
+  )
+  (label "+3V3" (at 143 40 0) (fields_autoplaced)
+    (effects (font (size 1.27 1.27)) (justify left)))
+  (label "GND" (at 143 40 0) (fields_autoplaced)
+    (effects (font (size 1.27 1.27)) (justify left)))
+  (label "PIEZO_PWM" (at 143 30 0) (fields_autoplaced)
+    (effects (font (size 1.27 1.27)) (justify left)))
+  (label "PIEZO_OUT" (at 143 37.5 0) (fields_autoplaced)
+    (effects (font (size 1.27 1.27)) (justify left)))
+  (label "PIEZO_RET" (at 143 37.5 0) (fields_autoplaced)
+    (effects (font (size 1.27 1.27)) (justify left)))
+  (symbol (lib_id "Device:R") (at 170 35 0) (unit 1)
+    (exclude_from_sim no) (in_bom yes) (on_board yes) (dnp no) (fields_autoplaced)
+    (property "Reference" "R7" (at 170 29 0)
+      (effects (font (size 1.27 1.27))))
+    (property "Value" "0R" (at 170 41 0)
+      (effects (font (size 1.27 1.27))))
+    (property "Footprint" "0402" (at 170 35 0)
+      (effects (font (size 1.27 1.27)) hide))
+    (property "Datasheet" "~" (at 170 35 0)
+      (effects (font (size 1.27 1.27)) hide))
+    (instances (project "card" (path "/card/sheets/audio" (reference "R7") (unit 1))))
+  )
+  (label "GND" (at 188 32.5 0) (fields_autoplaced)
+    (effects (font (size 1.27 1.27)) (justify left)))
+  (label "PIEZO_RET" (at 188 30 0) (fields_autoplaced)
+    (effects (font (size 1.27 1.27)) (justify left)))
+  (global_label "+3V3" (shape input) (at 280 20 0) (fields_autoplaced)
     (effects (font (size 1.27 1.27)) (justify left))
     (property "Intersheetrefs" "${INTERSHEET_REFS}" (at 280 20 0)
       (effects (font (size 1.27 1.27)) hide))
   )
-  (global_label "PIEZO_PWM" (shape input) (at 280 26 0) (fields_autoplaced)
+  (global_label "GND" (shape input) (at 280 26 0) (fields_autoplaced)
     (effects (font (size 1.27 1.27)) (justify left))
     (property "Intersheetrefs" "${INTERSHEET_REFS}" (at 280 26 0)
       (effects (font (size 1.27 1.27)) hide))
   )
+  (global_label "PIEZO_PWM" (shape input) (at 280 32 0) (fields_autoplaced)
+    (effects (font (size 1.27 1.27)) (justify left))
+    (property "Intersheetrefs" "${INTERSHEET_REFS}" (at 280 32 0)
+      (effects (font (size 1.27 1.27)) hide))
+  )
