File: hardware/card/schematic/sheets/controls.kicad_sch (KiCad schematic)
At the start: 12 parts, among them SW1 Tact, SW10A VolUp, SW10B VolDn, SW2 Tact, SW3 Tact, SW4 Tact, SW5 Tact, SW6 Tact, SW7 Tact, SW8 Tact, SW9 PowerPill

Commit message: pcb layout stuff
Parts:
- SW1, SW2, SW3, SW4, SW5, SW6, SW7, SW8: value Tact -> KMR211NG
- SW10A: value VolUp -> EVP-AKE31A
- SW10B: value VolDn -> EVP-AKE31A
- SW9: value PowerPill -> EVP-AKE31A
Changed lines of the file:
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@@
     (property "Reference" "SW1" (at 35 29 0)
       (effects (font (size 1.27 1.27))))
-    (property "Value" "Tact" (at 35 41 0)
+    (property "Value" "KMR211NG" (at 35 41 0)
       (effects (font (size 1.27 1.27))))
     (property "Footprint" "TBD" (at 35 35 0)
@@
     (property "Reference" "SW2" (at 80 29 0)
       (effects (font (size 1.27 1.27))))
-    (property "Value" "Tact" (at 80 41 0)
+    (property "Value" "KMR211NG" (at 80 41 0)
       (effects (font (size 1.27 1.27))))
     (property "Footprint" "TBD" (at 80 35 0)
@@
     (property "Reference" "SW3" (at 125 29 0)
       (effects (font (size 1.27 1.27))))
-    (property "Value" "Tact" (at 125 41 0)
+    (property "Value" "KMR211NG" (at 125 41 0)
       (effects (font (size 1.27 1.27))))
     (property "Footprint" "TBD" (at 125 35 0)
@@
     (property "Reference" "SW4" (at 170 29 0)
       (effects (font (size 1.27 1.27))))
-    (property "Value" "Tact" (at 170 41 0)
+    (property "Value" "KMR211NG" (at 170 41 0)
       (effects (font (size 1.27 1.27))))
     (property "Footprint" "TBD" (at 170 35 0)
@@
     (property "Reference" "SW5" (at 35 59 0)
       (effects (font (size 1.27 1.27))))
-    (property "Value" "Tact" (at 35 71 0)
+    (property "Value" "KMR211NG" (at 35 71 0)
       (effects (font (size 1.27 1.27))))
     (property "Footprint" "TBD" (at 35 65 0)
@@
     (property "Reference" "SW6" (at 80 59 0)
       (effects (font (size 1.27 1.27))))
-    (property "Value" "Tact" (at 80 71 0)
+    (property "Value" "KMR211NG" (at 80 71 0)
       (effects (font (size 1.27 1.27))))
     (property "Footprint" "TBD" (at 80 65 0)
@@
     (property "Reference" "SW7" (at 125 59 0)
       (effects (font (size 1.27 1.27))))
-    (property "Value" "Tact" (at 125 71 0)
+    (property "Value" "KMR211NG" (at 125 71 0)
       (effects (font (size 1.27 1.27))))
     (property "Footprint" "TBD" (at 125 65 0)
@@
     (property "Reference" "SW8" (at 170 59 0)
       (effects (font (size 1.27 1.27))))
-    (property "Value" "Tact" (at 170 71 0)
+    (property "Value" "KMR211NG" (at 170 71 0)
       (effects (font (size 1.27 1.27))))
     (property "Footprint" "TBD" (at 170 65 0)
@@
     (property "Reference" "SW9" (at 35 89 0)
       (effects (font (size 1.27 1.27))))
-    (property "Value" "PowerPill" (at 35 101 0)
+    (property "Value" "EVP-AKE31A" (at 35 101 0)
       (effects (font (size 1.27 1.27))))
     (property "Footprint" "TBD" (at 35 95 0)
@@
     (property "Reference" "SW10A" (at 80 89 0)
       (effects (font (size 1.27 1.27))))
-    (property "Value" "VolUp" (at 80 101 0)
+    (property "Value" "EVP-AKE31A" (at 80 101 0)
       (effects (font (size 1.27 1.27))))
     (property "Footprint" "TBD" (at 80 95 0)
@@
     (property "Reference" "SW10B" (at 125 89 0)
       (effects (font (size 1.27 1.27))))
-    (property "Value" "VolDn" (at 125 101 0)
+    (property "Value" "EVP-AKE31A" (at 125 101 0)
       (effects (font (size 1.27 1.27))))
     (property "Footprint" "TBD" (at 125 95 0)

Commit message: pcb stuff
Changed lines of the file:
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@@
     (instances (project "card" (path "/card/sheets/controls" (reference "SW9") (unit 1))))
   )
-  (label "ESP_EN" (at 53 92.5 0) (fields_autoplaced)
+  (label "GND" (at 53 92.5 0) (fields_autoplaced)
     (effects (font (size 1.27 1.27)) (justify left)))
   (label "SW_POWER" (at 53 90 0) (fields_autoplaced)
@@
       (effects (font (size 1.27 1.27)) hide))
   )
-  (global_label "ESP_EN" (shape input) (at 280 26 0) (fields_autoplaced)
+  (global_label "SW_DPAD_UP" (shape input) (at 280 26 0) (fields_autoplaced)
     (effects (font (size 1.27 1.27)) (justify left))
     (property "Intersheetrefs" "${INTERSHEET_REFS}" (at 280 26 0)
       (effects (font (size 1.27 1.27)) hide))
   )
-  (global_label "SW_DPAD_UP" (shape input) (at 280 32 0) (fields_autoplaced)
+  (global_label "SW_DPAD_DOWN" (shape input) (at 280 32 0) (fields_autoplaced)
     (effects (font (size 1.27 1.27)) (justify left))
     (property "Intersheetrefs" "${INTERSHEET_REFS}" (at 280 32 0)
       (effects (font (size 1.27 1.27)) hide))
   )
-  (global_label "SW_DPAD_DOWN" (shape input) (at 280 38 0) (fields_autoplaced)
+  (global_label "SW_DPAD_LEFT" (shape input) (at 280 38 0) (fields_autoplaced)
     (effects (font (size 1.27 1.27)) (justify left))
     (property "Intersheetrefs" "${INTERSHEET_REFS}" (at 280 38 0)
       (effects (font (size 1.27 1.27)) hide))
   )
-  (global_label "SW_DPAD_LEFT" (shape input) (at 280 44 0) (fields_autoplaced)
+  (global_label "SW_DPAD_RIGHT" (shape input) (at 280 44 0) (fields_autoplaced)
     (effects (font (size 1.27 1.27)) (justify left))
     (property "Intersheetrefs" "${INTERSHEET_REFS}" (at 280 44 0)
       (effects (font (size 1.27 1.27)) hide))
   )
-  (global_label "SW_DPAD_RIGHT" (shape input) (at 280 50 0) (fields_autoplaced)
+  (global_label "SW_ACTION" (shape input) (at 280 50 0) (fields_autoplaced)
     (effects (font (size 1.27 1.27)) (justify left))
     (property "Intersheetrefs" "${INTERSHEET_REFS}" (at 280 50 0)
       (effects (font (size 1.27 1.27)) hide))
   )
-  (global_label "SW_ACTION" (shape input) (at 280 56 0) (fields_autoplaced)
+  (global_label "SW_UNDO" (shape input) (at 280 56 0) (fields_autoplaced)
     (effects (font (size 1.27 1.27)) (justify left))
     (property "Intersheetrefs" "${INTERSHEET_REFS}" (at 280 56 0)
       (effects (font (size 1.27 1.27)) hide))
   )
-  (global_label "SW_UNDO" (shape input) (at 280 62 0) (fields_autoplaced)
+  (global_label "SW_RESTART" (shape input) (at 280 62 0) (fields_autoplaced)
     (effects (font (size 1.27 1.27)) (justify left))
     (property "Intersheetrefs" "${INTERSHEET_REFS}" (at 280 62 0)
       (effects (font (size 1.27 1.27)) hide))
   )
-  (global_label "SW_RESTART" (shape input) (at 280 68 0) (fields_autoplaced)
+  (global_label "SW_MENU" (shape input) (at 280 68 0) (fields_autoplaced)
     (effects (font (size 1.27 1.27)) (justify left))
     (property "Intersheetrefs" "${INTERSHEET_REFS}" (at 280 68 0)
       (effects (font (size 1.27 1.27)) hide))
   )
-  (global_label "SW_MENU" (shape input) (at 280 74 0) (fields_autoplaced)
+  (global_label "SW_POWER" (shape input) (at 280 74 0) (fields_autoplaced)
     (effects (font (size 1.27 1.27)) (justify left))
     (property "Intersheetrefs" "${INTERSHEET_REFS}" (at 280 74 0)
       (effects (font (size 1.27 1.27)) hide))
   )
-  (global_label "SW_POWER" (shape input) (at 280 80 0) (fields_autoplaced)
+  (global_label "VOL_UP" (shape input) (at 280 80 0) (fields_autoplaced)
     (effects (font (size 1.27 1.27)) (justify left))
     (property "Intersheetrefs" "${INTERSHEET_REFS}" (at 280 80 0)
       (effects (font (size 1.27 1.27)) hide))
   )
-  (global_label "VOL_UP" (shape input) (at 280 86 0) (fields_autoplaced)
+  (global_label "VOL_DOWN" (shape input) (at 280 86 0) (fields_autoplaced)
     (effects (font (size 1.27 1.27)) (justify left))
     (property "Intersheetrefs" "${INTERSHEET_REFS}" (at 280 86 0)
       (effects (font (size 1.27 1.27)) hide))
   )
-  (global_label "VOL_DOWN" (shape input) (at 280 20 0) (fields_autoplaced)
-    (effects (font (size 1.27 1.27)) (justify left))
-    (property "Intersheetrefs" "${INTERSHEET_REFS}" (at 280 20 0)
-      (effects (font (size 1.27 1.27)) hide))
-  )
