File: hardware/card/schematic/sheets/display.kicad_sch (KiCad schematic)
At the start: 2 parts, among them J3 FFC-15-1.0

Commit message: pcb layout stuff
Parts:
- J3: value FFC-15-1.0 -> FFC-15-1.0-FH12-class
Changed lines of the file:
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@@
     (property "Reference" "J3" (at 35 29 0)
       (effects (font (size 1.27 1.27))))
-    (property "Value" "FFC-15-1.0" (at 35 41 0)
+    (property "Value" "FFC-15-1.0-FH12-class" (at 35 41 0)
       (effects (font (size 1.27 1.27))))
     (property "Footprint" "TBD" (at 35 35 0)

Commit message: pcb stuff
Changed lines of the file:
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@@
     (instances (project "card" (path "/card/sheets/display" (reference "J3") (unit 1))))
   )
-  (label "+3V3" (at 53 32.5 0) (fields_autoplaced)
+  (label "+3V3_PANEL" (at 53 32.5 0) (fields_autoplaced)
     (effects (font (size 1.27 1.27)) (justify left)))
   (label "GND" (at 53 30 0) (fields_autoplaced)
@@
     (instances (project "card" (path "/card/sheets/display" (reference "C3") (unit 1))))
   )
-  (label "+3V3" (at 98 30 0) (fields_autoplaced)
+  (label "+3V3_PANEL" (at 98 30 0) (fields_autoplaced)
     (effects (font (size 1.27 1.27)) (justify left)))
   (label "GND" (at 98 32.5 0) (fields_autoplaced)
     (effects (font (size 1.27 1.27)) (justify left)))
-  (global_label "+3V3" (shape input) (at 280 20 0) (fields_autoplaced)
+  (global_label "+3V3_PANEL" (shape input) (at 280 20 0) (fields_autoplaced)
     (effects (font (size 1.27 1.27)) (justify left))
     (property "Intersheetrefs" "${INTERSHEET_REFS}" (at 280 20 0)
