File: hardware/card/schematic/sheets/haptic.kicad_sch (KiCad schematic)
At the start: 2 parts, among them U5 DRV2605L

Commit message: pcb layout stuff
Parts:
- B1: value LRA -> Coin-LRA-10mm
Changed lines of the file:
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@@
     (property "Reference" "B1" (at 80 29 0)
       (effects (font (size 1.27 1.27))))
-    (property "Value" "LRA" (at 80 41 0)
+    (property "Value" "Coin-LRA-10mm" (at 80 41 0)
       (effects (font (size 1.27 1.27))))
     (property "Footprint" "TBD" (at 80 35 0)
