File: hardware/card/schematic/sheets/power.kicad_sch (KiCad schematic)
At the start: 9 parts, among them J1 USB-C-mid, J2 Battery-JST, U2 BQ24075, U3 MAX17048, U4 TPS62135

Commit message: pcb layout stuff
Parts:
- J2: value Battery-JST -> 1S-Pouch-503048/603048
- U2: value BQ24075 -> BQ24075RGTR
- U3: value MAX17048 -> MAX17048G+T10
- U4: value TPS62135 -> TPS63070
Changed lines of the file:
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@@
     (property "Reference" "J2" (at 80 29 0)
       (effects (font (size 1.27 1.27))))
-    (property "Value" "Battery-JST" (at 80 41 0)
+    (property "Value" "1S-Pouch-503048/603048" (at 80 41 0)
       (effects (font (size 1.27 1.27))))
     (property "Footprint" "TBD" (at 80 35 0)
@@
     (property "Reference" "U2" (at 125 29 0)
       (effects (font (size 1.27 1.27))))
-    (property "Value" "BQ24075" (at 125 41 0)
+    (property "Value" "BQ24075RGTR" (at 125 41 0)
       (effects (font (size 1.27 1.27))))
     (property "Footprint" "TBD" (at 125 35 0)
@@
     (property "Reference" "U3" (at 170 29 0)
       (effects (font (size 1.27 1.27))))
-    (property "Value" "MAX17048" (at 170 41 0)
+    (property "Value" "MAX17048G+T10" (at 170 41 0)
       (effects (font (size 1.27 1.27))))
     (property "Footprint" "TBD" (at 170 35 0)
@@
     (property "Reference" "U4" (at 35 59 0)
       (effects (font (size 1.27 1.27))))
-    (property "Value" "TPS62135" (at 35 71 0)
+    (property "Value" "TPS63070" (at 35 71 0)
       (effects (font (size 1.27 1.27))))
     (property "Footprint" "TBD" (at 35 65 0)

Commit message: pcb stuff
Parts:
- added R1: 5.1k, 0402, symbol Device:R
- added U7: PowerLatch-DNP, TBD, symbol PSCard:Block2
- J2: value 1S-Pouch-503048/603048 -> 1S-Pouch-403048
- U6: renamed from R1; value 5.1k -> PanelLoadSwitch; footprint 0402 -> TBD; symbol Device:R -> PSCard:Block2
