File: hardware/card/schematic/sheets/debug.kicad_sch (KiCad schematic)
At the start: 4 parts

Commit message: hardware: replace U7 power latch with a slide switch (hard off)
Owner-approved power model: top-edge SPDT slide switch gates the TPS63070
EN pin; hard off is the normal off (Game Boy/Arduboy style, ~1-1.5 s tuned
cold boot, end-of-level atomic saves). Deletes the U7 latch IC and SYSOFF
wiring, frees GPIO8, adds a VBUS-powered charge LED on BQ24075 CHG, and
demotes deep sleep to an optional idle battery-saver. Closes the U7
pre-route gate from the 2026-07-09 PCB review.

Co-authored-by: Cursor <cursoragent@cursor.com>
Parts:
- removed TP4: EN, TestPoint, symbol PSCard:Block2
- added TP1: UART_TX, TestPoint, symbol PSCard:Block2
- TP2: renamed from TP1; value UART_TX -> UART_RX
- TP3: renamed from TP2; value UART_RX -> BOOT
- TP4: renamed from TP3; value BOOT -> EN
Other:
- moved on the sheet: TP2, TP3, TP4
Changed lines of the file:
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@@
   (title_block
     (title "PuzzleScript Card — debug")
-    (date "2026-07-08")
+    (date "2026-07-09")
     (rev "spin1")
     (comment 1 "Auto-generated from connectivity.json")
