File: hardware/card/easyeda_handoff/import/schematic/sheets/audio.kicad_sch (KiCad schematic)
At the start: 4 parts, among them Q1 NPN, U8 PiezoHBridge-DNP

Commit message: puzzlescript hardware case
Parts:
- JP1: footprint TBD -> TestPoint_Pad_D1.5mm
- Q1: footprint SOT23 -> SOT-23_L2.9-W1.6-P1.90-LS2.8-BR; LCSC (none) -> C94514; MPN (none) -> MMBT3904-7-F
- R7: footprint 0402 -> R0402; LCSC (none) -> C17168; MPN (none) -> 0402WGF0000TCE
- U8: footprint TBD -> W-QFN2020-12_L2.0-W2.0-P0.40-TL-EP0.9; LCSC (none) -> C510550; MPN (none) -> PAM8904EGPR
Changed lines of the file:
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@@
     (property "Value" "NPN" (at 35 41 0)
       (effects (font (size 1.27 1.27))))
-    (property "Footprint" "SOT23" (at 35 35 0)
+    (property "Footprint" "SOT-23_L2.9-W1.6-P1.90-LS2.8-BR" (at 35 35 0)
       (effects (font (size 1.27 1.27)) hide))
     (property "Datasheet" "~" (at 35 35 0)
+      (effects (font (size 1.27 1.27)) hide))
+    (property "LCSC" "C94514" (at 35 35 0)
+      (effects (font (size 1.27 1.27)) hide))
+    (property "MPN" "MMBT3904-7-F" (at 35 35 0)
       (effects (font (size 1.27 1.27)) hide))
     (instances (project "card" (path "/card/sheets/audio" (reference "Q1") (unit 1))))
@@
     (property "Value" "PiezoPads" (at 80 41 0)
       (effects (font (size 1.27 1.27))))
-    (property "Footprint" "TBD" (at 80 35 0)
+    (property "Footprint" "TestPoint_Pad_D1.5mm" (at 80 35 0)
       (effects (font (size 1.27 1.27)) hide))
     (property "Datasheet" "~" (at 80 35 0)
@@
     (property "Value" "PiezoHBridge-DNP" (at 125 41 0)
       (effects (font (size 1.27 1.27))))
-    (property "Footprint" "TBD" (at 125 35 0)
+    (property "Footprint" "W-QFN2020-12_L2.0-W2.0-P0.40-TL-EP0.9" (at 125 35 0)
       (effects (font (size 1.27 1.27)) hide))
     (property "Datasheet" "~" (at 125 35 0)
       (effects (font (size 1.27 1.27)) hide))
     (property "Gate" "GATE-PIEZO-DRIVE-REVIEW" (at 125 35 0)
+      (effects (font (size 1.27 1.27)) hide))
+    (property "LCSC" "C510550" (at 125 35 0)
+      (effects (font (size 1.27 1.27)) hide))
+    (property "MPN" "PAM8904EGPR" (at 125 35 0)
       (effects (font (size 1.27 1.27)) hide))
     (instances (project "card" (path "/card/sheets/audio" (reference "U8") (unit 1))))
@@
     (property "Value" "0R" (at 170 41 0)
       (effects (font (size 1.27 1.27))))
-    (property "Footprint" "0402" (at 170 35 0)
+    (property "Footprint" "R0402" (at 170 35 0)
       (effects (font (size 1.27 1.27)) hide))
     (property "Datasheet" "~" (at 170 35 0)
       (effects (font (size 1.27 1.27)) hide))
+    (property "LCSC" "C17168" (at 170 35 0)
+      (effects (font (size 1.27 1.27)) hide))
+    (property "MPN" "0402WGF0000TCE" (at 170 35 0)
+      (effects (font (size 1.27 1.27)) hide))
     (instances (project "card" (path "/card/sheets/audio" (reference "R7") (unit 1))))
