File: hardware/card/easyeda_handoff/import/schematic/sheets/compute.kicad_sch (KiCad schematic)
At the start: 8 parts, among them U1 ESP32-P4NRW32X, U9 QSPI-NOR-32MB, X1 40MHz-crystal

Commit message: puzzlescript hardware case
Parts:
- L1: value DCDC-inductor -> 2.2uH; footprint TBD -> IND-SMD_L4.0-W4.0_HPC4018BM; LCSC (none) -> C692155; MPN (none) -> HPC4018BM-2R2M
- R3, R4: footprint 0402 -> R0402; LCSC (none) -> C25900; MPN (none) -> 0402WGF4701TCE
- R5, R6: footprint 0402 -> R0402; LCSC (none) -> C25744; MPN (none) -> 0402WGF1002TCE
- U1: footprint QFN104-10x10-P0.35 -> QFN-104_L10.0-W10.0-P0.35-TL-EP7.5; LCSC (none) -> C22387510; MPN (none) -> ESP32-P4NRW32
- U9: footprint TBD -> WSON-8_L8.0-W6.10-P1.27-BL-EP; LCSC (none) -> C97522; MPN (none) -> W25Q256JVEIQ
- X1: footprint TBD -> SMD3225-4P; LCSC (none) -> C9010; MPN (none) -> X322540MPB4SI
Changed lines of the file:
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@@
     (property "Value" "ESP32-P4NRW32X" (at 35 41 0)
       (effects (font (size 1.27 1.27))))
-    (property "Footprint" "QFN104-10x10-P0.35" (at 35 35 0)
+    (property "Footprint" "QFN-104_L10.0-W10.0-P0.35-TL-EP7.5" (at 35 35 0)
       (effects (font (size 1.27 1.27)) hide))
     (property "Datasheet" "~" (at 35 35 0)
       (effects (font (size 1.27 1.27)) hide))
+    (property "LCSC" "C22387510" (at 35 35 0)
+      (effects (font (size 1.27 1.27)) hide))
+    (property "MPN" "ESP32-P4NRW32" (at 35 35 0)
+      (effects (font (size 1.27 1.27)) hide))
     (instances (project "card" (path "/card/sheets/compute" (reference "U1") (unit 1))))
   )
@@
     (property "Value" "QSPI-NOR-32MB" (at 80 41 0)
       (effects (font (size 1.27 1.27))))
-    (property "Footprint" "TBD" (at 80 35 0)
+    (property "Footprint" "WSON-8_L8.0-W6.10-P1.27-BL-EP" (at 80 35 0)
       (effects (font (size 1.27 1.27)) hide))
     (property "Datasheet" "~" (at 80 35 0)
@@
     (property "Gate" "GATE-ESP32-P4-REF-CAPTURE" (at 80 35 0)
       (effects (font (size 1.27 1.27)) hide))
+    (property "LCSC" "C97522" (at 80 35 0)
+      (effects (font (size 1.27 1.27)) hide))
+    (property "MPN" "W25Q256JVEIQ" (at 80 35 0)
+      (effects (font (size 1.27 1.27)) hide))
     (instances (project "card" (path "/card/sheets/compute" (reference "U9") (unit 1))))
   )
@@
     (property "Value" "40MHz-crystal" (at 125 41 0)
       (effects (font (size 1.27 1.27))))
-    (property "Footprint" "TBD" (at 125 35 0)
+    (property "Footprint" "SMD3225-4P" (at 125 35 0)
       (effects (font (size 1.27 1.27)) hide))
     (property "Datasheet" "~" (at 125 35 0)
@@
     (property "Gate" "GATE-ESP32-P4-REF-CAPTURE" (at 125 35 0)
       (effects (font (size 1.27 1.27)) hide))
+    (property "LCSC" "C9010" (at 125 35 0)
+      (effects (font (size 1.27 1.27)) hide))
+    (property "MPN" "X322540MPB4SI" (at 125 35 0)
+      (effects (font (size 1.27 1.27)) hide))
     (instances (project "card" (path "/card/sheets/compute" (reference "X1") (unit 1))))
   )
@@
     (property "Reference" "L1" (at 170 29 0)
       (effects (font (size 1.27 1.27))))
-    (property "Value" "DCDC-inductor" (at 170 41 0)
-      (effects (font (size 1.27 1.27))))
-    (property "Footprint" "TBD" (at 170 35 0)
+    (property "Value" "2.2uH" (at 170 41 0)
+      (effects (font (size 1.27 1.27))))
+    (property "Footprint" "IND-SMD_L4.0-W4.0_HPC4018BM" (at 170 35 0)
       (effects (font (size 1.27 1.27)) hide))
     (property "Datasheet" "~" (at 170 35 0)
@@
     (property "Gate" "GATE-ESP32-P4-REF-CAPTURE" (at 170 35 0)
       (effects (font (size 1.27 1.27)) hide))
+    (property "LCSC" "C692155" (at 170 35 0)
+      (effects (font (size 1.27 1.27)) hide))
+    (property "MPN" "HPC4018BM-2R2M" (at 170 35 0)
+      (effects (font (size 1.27 1.27)) hide))
     (instances (project "card" (path "/card/sheets/compute" (reference "L1") (unit 1))))
   )
@@
     (property "Value" "4.7k" (at 35 71 0)
       (effects (font (size 1.27 1.27))))
-    (property "Footprint" "0402" (at 35 65 0)
+    (property "Footprint" "R0402" (at 35 65 0)
       (effects (font (size 1.27 1.27)) hide))
     (property "Datasheet" "~" (at 35 65 0)
       (effects (font (size 1.27 1.27)) hide))
+    (property "LCSC" "C25900" (at 35 65 0)
+      (effects (font (size 1.27 1.27)) hide))
+    (property "MPN" "0402WGF4701TCE" (at 35 65 0)
+      (effects (font (size 1.27 1.27)) hide))
     (instances (project "card" (path "/card/sheets/compute" (reference "R3") (unit 1))))
   )
@@
     (property "Value" "4.7k" (at 80 71 0)
       (effects (font (size 1.27 1.27))))
-    (property "Footprint" "0402" (at 80 65 0)
+    (property "Footprint" "R0402" (at 80 65 0)
       (effects (font (size 1.27 1.27)) hide))
     (property "Datasheet" "~" (at 80 65 0)
       (effects (font (size 1.27 1.27)) hide))
+    (property "LCSC" "C25900" (at 80 65 0)
+      (effects (font (size 1.27 1.27)) hide))
+    (property "MPN" "0402WGF4701TCE" (at 80 65 0)
+      (effects (font (size 1.27 1.27)) hide))
     (instances (project "card" (path "/card/sheets/compute" (reference "R4") (unit 1))))
   )
@@
     (property "Value" "10k" (at 125 71 0)
       (effects (font (size 1.27 1.27))))
-    (property "Footprint" "0402" (at 125 65 0)
+    (property "Footprint" "R0402" (at 125 65 0)
       (effects (font (size 1.27 1.27)) hide))
     (property "Datasheet" "~" (at 125 65 0)
       (effects (font (size 1.27 1.27)) hide))
+    (property "LCSC" "C25744" (at 125 65 0)
+      (effects (font (size 1.27 1.27)) hide))
+    (property "MPN" "0402WGF1002TCE" (at 125 65 0)
+      (effects (font (size 1.27 1.27)) hide))
     (instances (project "card" (path "/card/sheets/compute" (reference "R5") (unit 1))))
   )
@@
     (property "Value" "10k" (at 170 71 0)
       (effects (font (size 1.27 1.27))))
-    (property "Footprint" "0402" (at 170 65 0)
+    (property "Footprint" "R0402" (at 170 65 0)
       (effects (font (size 1.27 1.27)) hide))
     (property "Datasheet" "~" (at 170 65 0)
       (effects (font (size 1.27 1.27)) hide))
+    (property "LCSC" "C25744" (at 170 65 0)
+      (effects (font (size 1.27 1.27)) hide))
+    (property "MPN" "0402WGF1002TCE" (at 170 65 0)
+      (effects (font (size 1.27 1.27)) hide))
     (instances (project "card" (path "/card/sheets/compute" (reference "R6") (unit 1))))
