File: hardware/card/easyeda_handoff/import/schematic/sheets/controls.kicad_sch (KiCad schematic)
At the start: 11 parts, among them SW1 TL3315NF160Q-class, SW10A EVP-AKE31A, SW10B EVP-AKE31A, SW2 TL3315NF160Q-class, SW3 TL3315NF160Q-class, SW4 TL3315NF160Q-class, SW5 KMR211NG, SW6 KMR211NG, SW7 KMR211NG, SW8 KMR211NG

Commit message: puzzlescript hardware case
Parts:
- R10: footprint 0402 -> R0402; LCSC (none) -> C25744; MPN (none) -> 0402WGF1002TCE
- SW1, SW2, SW3, SW4: footprint TBD -> SW-SMD_4P-L4.5-W4.5-P3.00-LS4.5-TL; LCSC (none) -> C2886877; MPN (none) -> TL3315NF160Q
- SW10A, SW10B: footprint EVPAK-side-push-3.9x2.9 -> SW-SMD_2P-L3.9-W2.9-P1.90-LS2.8-BR; LCSC (none) -> C569760; MPN (none) -> EVPAKE31A
- SW5, SW6, SW7, SW8: footprint TBD -> SW-SMD_4P-L6.0-W6.0-P4.50-LS6.5-TL; LCSC (none) -> C318438; MPN (none) -> KMR211NG LFS
Changed lines of the file:
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@@
     (property "Value" "TL3315NF160Q-class" (at 35 41 0)
       (effects (font (size 1.27 1.27))))
-    (property "Footprint" "TBD" (at 35 35 0)
+    (property "Footprint" "SW-SMD_4P-L4.5-W4.5-P3.00-LS4.5-TL" (at 35 35 0)
       (effects (font (size 1.27 1.27)) hide))
     (property "Datasheet" "~" (at 35 35 0)
@@
     (property "Gate" "GATE-DPAD-MOCKUP" (at 35 35 0)
       (effects (font (size 1.27 1.27)) hide))
+    (property "LCSC" "C2886877" (at 35 35 0)
+      (effects (font (size 1.27 1.27)) hide))
+    (property "MPN" "TL3315NF160Q" (at 35 35 0)
+      (effects (font (size 1.27 1.27)) hide))
     (instances (project "card" (path "/card/sheets/controls" (reference "SW1") (unit 1))))
   )
@@
     (property "Value" "TL3315NF160Q-class" (at 80 41 0)
       (effects (font (size 1.27 1.27))))
-    (property "Footprint" "TBD" (at 80 35 0)
+    (property "Footprint" "SW-SMD_4P-L4.5-W4.5-P3.00-LS4.5-TL" (at 80 35 0)
       (effects (font (size 1.27 1.27)) hide))
     (property "Datasheet" "~" (at 80 35 0)
@@
     (property "Gate" "GATE-DPAD-MOCKUP" (at 80 35 0)
       (effects (font (size 1.27 1.27)) hide))
+    (property "LCSC" "C2886877" (at 80 35 0)
+      (effects (font (size 1.27 1.27)) hide))
+    (property "MPN" "TL3315NF160Q" (at 80 35 0)
+      (effects (font (size 1.27 1.27)) hide))
     (instances (project "card" (path "/card/sheets/controls" (reference "SW2") (unit 1))))
   )
@@
     (property "Value" "TL3315NF160Q-class" (at 125 41 0)
       (effects (font (size 1.27 1.27))))
-    (property "Footprint" "TBD" (at 125 35 0)
+    (property "Footprint" "SW-SMD_4P-L4.5-W4.5-P3.00-LS4.5-TL" (at 125 35 0)
       (effects (font (size 1.27 1.27)) hide))
     (property "Datasheet" "~" (at 125 35 0)
@@
     (property "Gate" "GATE-DPAD-MOCKUP" (at 125 35 0)
       (effects (font (size 1.27 1.27)) hide))
+    (property "LCSC" "C2886877" (at 125 35 0)
+      (effects (font (size 1.27 1.27)) hide))
+    (property "MPN" "TL3315NF160Q" (at 125 35 0)
+      (effects (font (size 1.27 1.27)) hide))
     (instances (project "card" (path "/card/sheets/controls" (reference "SW3") (unit 1))))
   )
@@
     (property "Value" "TL3315NF160Q-class" (at 170 41 0)
       (effects (font (size 1.27 1.27))))
-    (property "Footprint" "TBD" (at 170 35 0)
+    (property "Footprint" "SW-SMD_4P-L4.5-W4.5-P3.00-LS4.5-TL" (at 170 35 0)
       (effects (font (size 1.27 1.27)) hide))
     (property "Datasheet" "~" (at 170 35 0)
@@
     (property "Gate" "GATE-DPAD-MOCKUP" (at 170 35 0)
       (effects (font (size 1.27 1.27)) hide))
+    (property "LCSC" "C2886877" (at 170 35 0)
+      (effects (font (size 1.27 1.27)) hide))
+    (property "MPN" "TL3315NF160Q" (at 170 35 0)
+      (effects (font (size 1.27 1.27)) hide))
     (instances (project "card" (path "/card/sheets/controls" (reference "SW4") (unit 1))))
   )
@@
     (property "Value" "KMR211NG" (at 35 71 0)
       (effects (font (size 1.27 1.27))))
-    (property "Footprint" "TBD" (at 35 65 0)
+    (property "Footprint" "SW-SMD_4P-L6.0-W6.0-P4.50-LS6.5-TL" (at 35 65 0)
       (effects (font (size 1.27 1.27)) hide))
     (property "Datasheet" "~" (at 35 65 0)
@@
     (property "Gate" "GATE-FACE-BUTTON-FEEL" (at 35 65 0)
       (effects (font (size 1.27 1.27)) hide))
+    (property "LCSC" "C318438" (at 35 65 0)
+      (effects (font (size 1.27 1.27)) hide))
+    (property "MPN" "KMR211NG LFS" (at 35 65 0)
+      (effects (font (size 1.27 1.27)) hide))
     (instances (project "card" (path "/card/sheets/controls" (reference "SW5") (unit 1))))
   )
@@
     (property "Value" "KMR211NG" (at 80 71 0)
       (effects (font (size 1.27 1.27))))
-    (property "Footprint" "TBD" (at 80 65 0)
+    (property "Footprint" "SW-SMD_4P-L6.0-W6.0-P4.50-LS6.5-TL" (at 80 65 0)
       (effects (font (size 1.27 1.27)) hide))
     (property "Datasheet" "~" (at 80 65 0)
@@
     (property "Gate" "GATE-FACE-BUTTON-FEEL" (at 80 65 0)
       (effects (font (size 1.27 1.27)) hide))
+    (property "LCSC" "C318438" (at 80 65 0)
+      (effects (font (size 1.27 1.27)) hide))
+    (property "MPN" "KMR211NG LFS" (at 80 65 0)
+      (effects (font (size 1.27 1.27)) hide))
     (instances (project "card" (path "/card/sheets/controls" (reference "SW6") (unit 1))))
   )
@@
     (property "Value" "KMR211NG" (at 125 71 0)
       (effects (font (size 1.27 1.27))))
-    (property "Footprint" "TBD" (at 125 65 0)
+    (property "Footprint" "SW-SMD_4P-L6.0-W6.0-P4.50-LS6.5-TL" (at 125 65 0)
       (effects (font (size 1.27 1.27)) hide))
     (property "Datasheet" "~" (at 125 65 0)
@@
     (property "Gate" "GATE-FACE-BUTTON-FEEL" (at 125 65 0)
       (effects (font (size 1.27 1.27)) hide))
+    (property "LCSC" "C318438" (at 125 65 0)
+      (effects (font (size 1.27 1.27)) hide))
+    (property "MPN" "KMR211NG LFS" (at 125 65 0)
+      (effects (font (size 1.27 1.27)) hide))
     (instances (project "card" (path "/card/sheets/controls" (reference "SW7") (unit 1))))
   )
@@
     (property "Value" "KMR211NG" (at 170 71 0)
       (effects (font (size 1.27 1.27))))
-    (property "Footprint" "TBD" (at 170 65 0)
+    (property "Footprint" "SW-SMD_4P-L6.0-W6.0-P4.50-LS6.5-TL" (at 170 65 0)
       (effects (font (size 1.27 1.27)) hide))
     (property "Datasheet" "~" (at 170 65 0)
@@
     (property "Gate" "GATE-FACE-BUTTON-FEEL" (at 170 65 0)
       (effects (font (size 1.27 1.27)) hide))
+    (property "LCSC" "C318438" (at 170 65 0)
+      (effects (font (size 1.27 1.27)) hide))
+    (property "MPN" "KMR211NG LFS" (at 170 65 0)
+      (effects (font (size 1.27 1.27)) hide))
     (instances (project "card" (path "/card/sheets/controls" (reference "SW8") (unit 1))))
   )
@@
     (property "Value" "EVP-AKE31A" (at 35 101 0)
       (effects (font (size 1.27 1.27))))
-    (property "Footprint" "EVPAK-side-push-3.9x2.9" (at 35 95 0)
+    (property "Footprint" "SW-SMD_2P-L3.9-W2.9-P1.90-LS2.8-BR" (at 35 95 0)
       (effects (font (size 1.27 1.27)) hide))
     (property "Datasheet" "~" (at 35 95 0)
       (effects (font (size 1.27 1.27)) hide))
+    (property "LCSC" "C569760" (at 35 95 0)
+      (effects (font (size 1.27 1.27)) hide))
+    (property "MPN" "EVPAKE31A" (at 35 95 0)
+      (effects (font (size 1.27 1.27)) hide))
     (instances (project "card" (path "/card/sheets/controls" (reference "SW10A") (unit 1))))
   )
@@
     (property "Value" "EVP-AKE31A" (at 80 101 0)
       (effects (font (size 1.27 1.27))))
-    (property "Footprint" "EVPAK-side-push-3.9x2.9" (at 80 95 0)
+    (property "Footprint" "SW-SMD_2P-L3.9-W2.9-P1.90-LS2.8-BR" (at 80 95 0)
       (effects (font (size 1.27 1.27)) hide))
     (property "Datasheet" "~" (at 80 95 0)
       (effects (font (size 1.27 1.27)) hide))
+    (property "LCSC" "C569760" (at 80 95 0)
+      (effects (font (size 1.27 1.27)) hide))
+    (property "MPN" "EVPAKE31A" (at 80 95 0)
+      (effects (font (size 1.27 1.27)) hide))
     (instances (project "card" (path "/card/sheets/controls" (reference "SW10B") (unit 1))))
   )
@@
     (property "Value" "10k" (at 125 101 0)
       (effects (font (size 1.27 1.27))))
-    (property "Footprint" "0402" (at 125 95 0)
+    (property "Footprint" "R0402" (at 125 95 0)
       (effects (font (size 1.27 1.27)) hide))
     (property "Datasheet" "~" (at 125 95 0)
       (effects (font (size 1.27 1.27)) hide))
+    (property "LCSC" "C25744" (at 125 95 0)
+      (effects (font (size 1.27 1.27)) hide))
+    (property "MPN" "0402WGF1002TCE" (at 125 95 0)
+      (effects (font (size 1.27 1.27)) hide))
     (instances (project "card" (path "/card/sheets/controls" (reference "R10") (unit 1))))
