File: hardware/card/easyeda_handoff/import/schematic/sheets/display.kicad_sch (KiCad schematic)
At the start: 2 parts, among them J3 FFC-15-1.0-FH12-class

Commit message: puzzlescript hardware case
Parts:
- C3: footprint 0603 -> C0603; LCSC (none) -> C19702; MPN (none) -> CL10A106KP8NNNC
- J3: footprint FFC-15-1.0mm-right-angle-contact-TBD -> FPC-SMD_FH12-15S-0.5SH-55; LCSC (none) -> C2832207; MPN (none) -> FH12-15S-0.5SH(55)
Changed lines of the file:
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@@
     (property "Value" "FFC-15-1.0-FH12-class" (at 35 41 0)
       (effects (font (size 1.27 1.27))))
-    (property "Footprint" "FFC-15-1.0mm-right-angle-contact-TBD" (at 35 35 0)
+    (property "Footprint" "FPC-SMD_FH12-15S-0.5SH-55" (at 35 35 0)
       (effects (font (size 1.27 1.27)) hide))
     (property "Datasheet" "~" (at 35 35 0)
       (effects (font (size 1.27 1.27)) hide))
     (property "Gate" "GATE-DSI-FFC-CONTACT" (at 35 35 0)
+      (effects (font (size 1.27 1.27)) hide))
+    (property "LCSC" "C2832207" (at 35 35 0)
+      (effects (font (size 1.27 1.27)) hide))
+    (property "MPN" "FH12-15S-0.5SH(55)" (at 35 35 0)
       (effects (font (size 1.27 1.27)) hide))
     (instances (project "card" (path "/card/sheets/display" (reference "J3") (unit 1))))
@@
     (property "Value" "10u" (at 80 41 0)
       (effects (font (size 1.27 1.27))))
-    (property "Footprint" "0603" (at 80 35 0)
+    (property "Footprint" "C0603" (at 80 35 0)
       (effects (font (size 1.27 1.27)) hide))
     (property "Datasheet" "~" (at 80 35 0)
       (effects (font (size 1.27 1.27)) hide))
+    (property "LCSC" "C19702" (at 80 35 0)
+      (effects (font (size 1.27 1.27)) hide))
+    (property "MPN" "CL10A106KP8NNNC" (at 80 35 0)
+      (effects (font (size 1.27 1.27)) hide))
     (instances (project "card" (path "/card/sheets/display" (reference "C3") (unit 1))))
