File: hardware/card/easyeda_handoff/import/schematic/sheets/haptic.kicad_sch (KiCad schematic)
At the start: 2 parts, among them U5 DRV2605LDGS

Commit message: puzzlescript hardware case
Parts:
- B1: footprint TBD -> VIBRATING-MOTOR-SMD_WELDING; LCSC (none) -> C2759984; MPN (none) -> LCM1027A2445F
- U5: footprint VSSOP-10-DGS-3x4.9 -> VSSOP-10_L3.0-W3.0-P0.50-LS4.9-BL; LCSC (none) -> C527464; MPN (none) -> DRV2605LDGSR
Changed lines of the file:
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@@
     (property "Value" "DRV2605LDGS" (at 35 41 0)
       (effects (font (size 1.27 1.27))))
-    (property "Footprint" "VSSOP-10-DGS-3x4.9" (at 35 35 0)
+    (property "Footprint" "VSSOP-10_L3.0-W3.0-P0.50-LS4.9-BL" (at 35 35 0)
       (effects (font (size 1.27 1.27)) hide))
     (property "Datasheet" "~" (at 35 35 0)
+      (effects (font (size 1.27 1.27)) hide))
+    (property "LCSC" "C527464" (at 35 35 0)
+      (effects (font (size 1.27 1.27)) hide))
+    (property "MPN" "DRV2605LDGSR" (at 35 35 0)
       (effects (font (size 1.27 1.27)) hide))
     (instances (project "card" (path "/card/sheets/haptic" (reference "U5") (unit 1))))
@@
     (property "Value" "Coin-LRA-10mm" (at 80 41 0)
       (effects (font (size 1.27 1.27))))
-    (property "Footprint" "TBD" (at 80 35 0)
+    (property "Footprint" "VIBRATING-MOTOR-SMD_WELDING" (at 80 35 0)
       (effects (font (size 1.27 1.27)) hide))
     (property "Datasheet" "~" (at 80 35 0)
@@
     (property "Gate" "GATE-LRA-MOUNT" (at 80 35 0)
       (effects (font (size 1.27 1.27)) hide))
+    (property "LCSC" "C2759984" (at 80 35 0)
+      (effects (font (size 1.27 1.27)) hide))
+    (property "MPN" "LCM1027A2445F" (at 80 35 0)
+      (effects (font (size 1.27 1.27)) hide))
     (instances (project "card" (path "/card/sheets/haptic" (reference "B1") (unit 1))))
