File: hardware/card/easyeda_handoff/import/schematic/sheets/led.kicad_sch (KiCad schematic)
At the start: 3 parts

Commit message: puzzlescript hardware case
Parts:
- D1: footprint TBD -> LED0603-RD; LCSC (none) -> C72043; MPN (none) -> 19-217/GHC-YR1S2/3T
- D2: footprint TBD -> LED0603-GN; LCSC (none) -> C2290; MPN (none) -> 19-217/GCT-CB2C6SG1/3T
- D3: footprint TBD -> LED0603-FD_BLUE; LCSC (none) -> C72041; MPN (none) -> 19-217/BHC-ZL1M2RY/3T
Changed lines of the file:
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@@
     (property "Value" "LED-R" (at 35 41 0)
       (effects (font (size 1.27 1.27))))
-    (property "Footprint" "TBD" (at 35 35 0)
+    (property "Footprint" "LED0603-RD" (at 35 35 0)
       (effects (font (size 1.27 1.27)) hide))
     (property "Datasheet" "~" (at 35 35 0)
       (effects (font (size 1.27 1.27)) hide))
     (property "Gate" "GATE-CASE-LED-LIGHTPIPE" (at 35 35 0)
+      (effects (font (size 1.27 1.27)) hide))
+    (property "LCSC" "C72043" (at 35 35 0)
+      (effects (font (size 1.27 1.27)) hide))
+    (property "MPN" "19-217/GHC-YR1S2/3T" (at 35 35 0)
       (effects (font (size 1.27 1.27)) hide))
     (instances (project "card" (path "/card/sheets/led" (reference "D1") (unit 1))))
@@
     (property "Value" "LED-G" (at 80 41 0)
       (effects (font (size 1.27 1.27))))
-    (property "Footprint" "TBD" (at 80 35 0)
+    (property "Footprint" "LED0603-GN" (at 80 35 0)
       (effects (font (size 1.27 1.27)) hide))
     (property "Datasheet" "~" (at 80 35 0)
       (effects (font (size 1.27 1.27)) hide))
     (property "Gate" "GATE-CASE-LED-LIGHTPIPE" (at 80 35 0)
+      (effects (font (size 1.27 1.27)) hide))
+    (property "LCSC" "C2290" (at 80 35 0)
+      (effects (font (size 1.27 1.27)) hide))
+    (property "MPN" "19-217/GCT-CB2C6SG1/3T" (at 80 35 0)
       (effects (font (size 1.27 1.27)) hide))
     (instances (project "card" (path "/card/sheets/led" (reference "D2") (unit 1))))
@@
     (property "Value" "LED-B" (at 125 41 0)
       (effects (font (size 1.27 1.27))))
-    (property "Footprint" "TBD" (at 125 35 0)
+    (property "Footprint" "LED0603-FD_BLUE" (at 125 35 0)
       (effects (font (size 1.27 1.27)) hide))
     (property "Datasheet" "~" (at 125 35 0)
@@
     (property "Gate" "GATE-CASE-LED-LIGHTPIPE" (at 125 35 0)
       (effects (font (size 1.27 1.27)) hide))
+    (property "LCSC" "C72041" (at 125 35 0)
+      (effects (font (size 1.27 1.27)) hide))
+    (property "MPN" "19-217/BHC-ZL1M2RY/3T" (at 125 35 0)
+      (effects (font (size 1.27 1.27)) hide))
     (instances (project "card" (path "/card/sheets/led" (reference "D3") (unit 1))))
