File: hardware/card/easyeda_handoff/import/schematic/sheets/power.kicad_sch (KiCad schematic)
At the start: 13 parts, among them J1 HRO-TYPE-C-31-M-12, J2 1S-Pouch-403048, SW9 SlideSwitch-SPDT-JS102000-cla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, U2 BQ24075RGTR, U3 MAX17048G+T10, U4 TPS63070, U6 TPS22919DCK

Commit message: puzzlescript hardware case
Parts:
- C1, C2: footprint 0603 -> C0603; LCSC (none) -> C19702; MPN (none) -> CL10A106KP8NNNC
- D4: footprint 0603 -> LED0603-RD; LCSC (none) -> C72043; MPN (none) -> 19-217/GHC-YR1S2/3T
- J1: footprint Connector_USB:USB_C_Receptacle_HRO_TYPE-C-31-M-12 -> USB-C-SMD_TYPE-C-16PIN-2MD-073; LCSC (none) -> C2765186; MPN (none) -> TYPE-C 16PIN 2MD(073)
- J2: footprint TBD -> CONN-SMD_SM02B-SRSS-TB; LCSC (none) -> C160404; MPN (none) -> SM02B-SRSS-TB(LF)(SN)
- R1, R2: footprint 0402 -> R0402; LCSC (none) -> C25905; MPN (none) -> 0402WGF5101TCE
- R8: footprint 0402 -> R0402; LCSC (none) -> C11702; MPN (none) -> 0402WGF1001TCE
- SW9: footprint TBD -> SW-SMD_6P-L7.0-W3.5-P1.27-LS4.5-TL; LCSC (none) -> C431544; MPN (none) -> JS102011SAQN
- U2: footprint VQFN-16-RGT-3x3 -> QFN-16_L3.0-W3.0-P0.50-TL-EP1.7; LCSC (none) -> C15464; MPN (none) -> BQ24075RGTR
- U3: footprint LFCSP-8-2x2 -> TDFN-8_L2.0-W2.0-P0.50-BL-EP1.2; LCSC (none) -> C2682616; MPN (none) -> MAX17048G+T10
- U4: footprint VQFN-HR-15-RNM-3x2.5 -> VQFN-HR-15_L3.0-W2.5-P0.50-BL_TPS63070RNMR; LCSC (none) -> C964639; MPN (none) -> TPS63070RNMT
- U6: footprint SOT-SC70-6-DCK-2x2.1 -> SC-70-6_L2.2-W1.3-P0.65-LS2.1-BR; LCSC (none) -> C2149796; MPN (none) -> TPS22919DCKR
Changed lines of the file:
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@@
     (property "Value" "HRO-TYPE-C-31-M-12" (at 35 41 0)
       (effects (font (size 1.27 1.27))))
-    (property "Footprint" "Connector_USB:USB_C_Receptacle_HRO_TYPE-C-31-M-12" (at 35 35 0)
+    (property "Footprint" "USB-C-SMD_TYPE-C-16PIN-2MD-073" (at 35 35 0)
       (effects (font (size 1.27 1.27)) hide))
     (property "Datasheet" "~" (at 35 35 0)
       (effects (font (size 1.27 1.27)) hide))
+    (property "LCSC" "C2765186" (at 35 35 0)
+      (effects (font (size 1.27 1.27)) hide))
+    (property "MPN" "TYPE-C 16PIN 2MD(073)" (at 35 35 0)
+      (effects (font (size 1.27 1.27)) hide))
     (instances (project "card" (path "/card/sheets/power" (reference "J1") (unit 1))))
   )
@@
     (property "Value" "1S-Pouch-403048" (at 80 41 0)
       (effects (font (size 1.27 1.27))))
-    (property "Footprint" "TBD" (at 80 35 0)
+    (property "Footprint" "CONN-SMD_SM02B-SRSS-TB" (at 80 35 0)
       (effects (font (size 1.27 1.27)) hide))
     (property "Datasheet" "~" (at 80 35 0)
@@
     (property "Gate" "GATE-BATTERY-SAMPLE" (at 80 35 0)
       (effects (font (size 1.27 1.27)) hide))
+    (property "LCSC" "C160404" (at 80 35 0)
+      (effects (font (size 1.27 1.27)) hide))
+    (property "MPN" "SM02B-SRSS-TB(LF)(SN)" (at 80 35 0)
+      (effects (font (size 1.27 1.27)) hide))
     (instances (project "card" (path "/card/sheets/power" (reference "J2") (unit 1))))
   )
@@
     (property "Value" "BQ24075RGTR" (at 125 41 0)
       (effects (font (size 1.27 1.27))))
-    (property "Footprint" "VQFN-16-RGT-3x3" (at 125 35 0)
+    (property "Footprint" "QFN-16_L3.0-W3.0-P0.50-TL-EP1.7" (at 125 35 0)
       (effects (font (size 1.27 1.27)) hide))
     (property "Datasheet" "~" (at 125 35 0)
       (effects (font (size 1.27 1.27)) hide))
+    (property "LCSC" "C15464" (at 125 35 0)
+      (effects (font (size 1.27 1.27)) hide))
+    (property "MPN" "BQ24075RGTR" (at 125 35 0)
+      (effects (font (size 1.27 1.27)) hide))
     (instances (project "card" (path "/card/sheets/power" (reference "U2") (unit 1))))
   )
@@
     (property "Value" "MAX17048G+T10" (at 170 41 0)
       (effects (font (size 1.27 1.27))))
-    (property "Footprint" "LFCSP-8-2x2" (at 170 35 0)
+    (property "Footprint" "TDFN-8_L2.0-W2.0-P0.50-BL-EP1.2" (at 170 35 0)
       (effects (font (size 1.27 1.27)) hide))
     (property "Datasheet" "~" (at 170 35 0)
       (effects (font (size 1.27 1.27)) hide))
+    (property "LCSC" "C2682616" (at 170 35 0)
+      (effects (font (size 1.27 1.27)) hide))
+    (property "MPN" "MAX17048G+T10" (at 170 35 0)
+      (effects (font (size 1.27 1.27)) hide))
     (instances (project "card" (path "/card/sheets/power" (reference "U3") (unit 1))))
   )
@@
     (property "Value" "TPS63070" (at 35 71 0)
       (effects (font (size 1.27 1.27))))
-    (property "Footprint" "VQFN-HR-15-RNM-3x2.5" (at 35 65 0)
+    (property "Footprint" "VQFN-HR-15_L3.0-W2.5-P0.50-BL_TPS63070RNMR" (at 35 65 0)
       (effects (font (size 1.27 1.27)) hide))
     (property "Datasheet" "~" (at 35 65 0)
       (effects (font (size 1.27 1.27)) hide))
+    (property "LCSC" "C964639" (at 35 65 0)
+      (effects (font (size 1.27 1.27)) hide))
+    (property "MPN" "TPS63070RNMT" (at 35 65 0)
+      (effects (font (size 1.27 1.27)) hide))
     (instances (project "card" (path "/card/sheets/power" (reference "U4") (unit 1))))
   )
@@
     (property "Value" "TPS22919DCK" (at 80 71 0)
       (effects (font (size 1.27 1.27))))
-    (property "Footprint" "SOT-SC70-6-DCK-2x2.1" (at 80 65 0)
+    (property "Footprint" "SC-70-6_L2.2-W1.3-P0.65-LS2.1-BR" (at 80 65 0)
       (effects (font (size 1.27 1.27)) hide))
     (property "Datasheet" "~" (at 80 65 0)
       (effects (font (size 1.27 1.27)) hide))
+    (property "LCSC" "C2149796" (at 80 65 0)
+      (effects (font (size 1.27 1.27)) hide))
+    (property "MPN" "TPS22919DCKR" (at 80 65 0)
+      (effects (font (size 1.27 1.27)) hide))
     (instances (project "card" (path "/card/sheets/power" (reference "U6") (unit 1))))
   )
@@
     (property "Value" "SlideSwitch-SPDT-JS102000-class" (at 125 71 0)
       (effects (font (size 1.27 1.27))))
-    (property "Footprint" "TBD" (at 125 65 0)
+    (property "Footprint" "SW-SMD_6P-L7.0-W3.5-P1.27-LS4.5-TL" (at 125 65 0)
       (effects (font (size 1.27 1.27)) hide))
     (property "Datasheet" "~" (at 125 65 0)
@@
     (property "Gate" "GATE-POWER-SLIDE-SLOT" (at 125 65 0)
       (effects (font (size 1.27 1.27)) hide))
+    (property "LCSC" "C431544" (at 125 65 0)
+      (effects (font (size 1.27 1.27)) hide))
+    (property "MPN" "JS102011SAQN" (at 125 65 0)
+      (effects (font (size 1.27 1.27)) hide))
     (instances (project "card" (path "/card/sheets/power" (reference "SW9") (unit 1))))
   )
@@
     (property "Value" "LED-CHG" (at 170 71 0)
       (effects (font (size 1.27 1.27))))
-    (property "Footprint" "0603" (at 170 65 0)
+    (property "Footprint" "LED0603-RD" (at 170 65 0)
       (effects (font (size 1.27 1.27)) hide))
     (property "Datasheet" "~" (at 170 65 0)
       (effects (font (size 1.27 1.27)) hide))
+    (property "LCSC" "C72043" (at 170 65 0)
+      (effects (font (size 1.27 1.27)) hide))
+    (property "MPN" "19-217/GHC-YR1S2/3T" (at 170 65 0)
+      (effects (font (size 1.27 1.27)) hide))
     (instances (project "card" (path "/card/sheets/power" (reference "D4") (unit 1))))
   )
@@
     (property "Value" "1k" (at 35 101 0)
       (effects (font (size 1.27 1.27))))
-    (property "Footprint" "0402" (at 35 95 0)
+    (property "Footprint" "R0402" (at 35 95 0)
       (effects (font (size 1.27 1.27)) hide))
     (property "Datasheet" "~" (at 35 95 0)
       (effects (font (size 1.27 1.27)) hide))
+    (property "LCSC" "C11702" (at 35 95 0)
+      (effects (font (size 1.27 1.27)) hide))
+    (property "MPN" "0402WGF1001TCE" (at 35 95 0)
+      (effects (font (size 1.27 1.27)) hide))
     (instances (project "card" (path "/card/sheets/power" (reference "R8") (unit 1))))
   )
@@
     (property "Value" "5.1k" (at 80 101 0)
       (effects (font (size 1.27 1.27))))
-    (property "Footprint" "0402" (at 80 95 0)
+    (property "Footprint" "R0402" (at 80 95 0)
       (effects (font (size 1.27 1.27)) hide))
     (property "Datasheet" "~" (at 80 95 0)
       (effects (font (size 1.27 1.27)) hide))
+    (property "LCSC" "C25905" (at 80 95 0)
+      (effects (font (size 1.27 1.27)) hide))
+    (property "MPN" "0402WGF5101TCE" (at 80 95 0)
+      (effects (font (size 1.27 1.27)) hide))
     (instances (project "card" (path "/card/sheets/power" (reference "R1") (unit 1))))
   )
@@
     (property "Value" "5.1k" (at 125 101 0)
       (effects (font (size 1.27 1.27))))
-    (property "Footprint" "0402" (at 125 95 0)
+    (property "Footprint" "R0402" (at 125 95 0)
       (effects (font (size 1.27 1.27)) hide))
     (property "Datasheet" "~" (at 125 95 0)
       (effects (font (size 1.27 1.27)) hide))
+    (property "LCSC" "C25905" (at 125 95 0)
+      (effects (font (size 1.27 1.27)) hide))
+    (property "MPN" "0402WGF5101TCE" (at 125 95 0)
+      (effects (font (size 1.27 1.27)) hide))
     (instances (project "card" (path "/card/sheets/power" (reference "R2") (unit 1))))
   )
@@
     (property "Value" "10u" (at 170 101 0)
       (effects (font (size 1.27 1.27))))
-    (property "Footprint" "0603" (at 170 95 0)
+    (property "Footprint" "C0603" (at 170 95 0)
       (effects (font (size 1.27 1.27)) hide))
     (property "Datasheet" "~" (at 170 95 0)
       (effects (font (size 1.27 1.27)) hide))
+    (property "LCSC" "C19702" (at 170 95 0)
+      (effects (font (size 1.27 1.27)) hide))
+    (property "MPN" "CL10A106KP8NNNC" (at 170 95 0)
+      (effects (font (size 1.27 1.27)) hide))
     (instances (project "card" (path "/card/sheets/power" (reference "C1") (unit 1))))
   )
@@
     (property "Value" "10u" (at 35 131 0)
       (effects (font (size 1.27 1.27))))
-    (property "Footprint" "0603" (at 35 125 0)
+    (property "Footprint" "C0603" (at 35 125 0)
       (effects (font (size 1.27 1.27)) hide))
     (property "Datasheet" "~" (at 35 125 0)
       (effects (font (size 1.27 1.27)) hide))
+    (property "LCSC" "C19702" (at 35 125 0)
+      (effects (font (size 1.27 1.27)) hide))
+    (property "MPN" "CL10A106KP8NNNC" (at 35 125 0)
+      (effects (font (size 1.27 1.27)) hide))
     (instances (project "card" (path "/card/sheets/power" (reference "C2") (unit 1))))
