File: hardware/card/easyeda_handoff/import/schematic/sheets/storage.kicad_sch (KiCad schematic)
At the start: 1 part, among them J4 microSD

Commit message: puzzlescript hardware case
Parts:
- J4: footprint TBD -> TF-015; LCSC (none) -> C113206; MPN (none) -> TF-015
Changed lines of the file:
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@@
     (property "Value" "microSD" (at 35 41 0)
       (effects (font (size 1.27 1.27))))
-    (property "Footprint" "TBD" (at 35 35 0)
+    (property "Footprint" "TF-015" (at 35 35 0)
       (effects (font (size 1.27 1.27)) hide))
     (property "Datasheet" "~" (at 35 35 0)
@@
     (property "Gate" "GATE-MICROSD-FOOTPRINT" (at 35 35 0)
       (effects (font (size 1.27 1.27)) hide))
+    (property "LCSC" "C113206" (at 35 35 0)
+      (effects (font (size 1.27 1.27)) hide))
+    (property "MPN" "TF-015" (at 35 35 0)
+      (effects (font (size 1.27 1.27)) hide))
     (instances (project "card" (path "/card/sheets/storage" (reference "J4") (unit 1))))
