File: hardware/pocket_card/case/out/pcb/pocket_card_controller.kicad_pcb (KiCad board)
At the start: 2 copper layers, 80.5 x 37 mm, 19 parts, among them U1 SOIC-28W_7.5x17.9mm_P1.27mm

Commit message: Use a top-actuated tact switch; the buttons were side-push parts
Every button footprint was Panasonic_EVQPUJ_EVQPUA, which is a SIDE-actuated
switch: 6.40 x 4.50 x 1.65, no plunger anywhere on its top face, and its body
offset in y where the side actuator protrudes. The caps press straight down onto
a face that does not actuate, so not one of the eight buttons would have worked.

Nothing electrical could have caught it. The pad layouts are nearly identical --
+/-2.62 x +/-0.85 against +/-2.58 x +/-0.85 -- so netlist, DRC and routing were
all perfectly happy. It was visible only in KiCad's 3D view.

Now SW_SPST_EVQP2_MiddlePushTravel_H2.5mm: top-actuated, 2.50 mm tall, which is
what TACT_H already claimed, with a centred 1.8 x 1.8 plunger for the cap boss
to press. Verified by measuring the STEP models rather than reading names.
TACT_H is promoted from DECIDED to DATASHEET; travel and force stay ASSUMED,
since EVQ-P2 ships in several variants and neither has been read off a datasheet.

Board rebuilt: unconnected 10 -> 4, violations 30 -> 25.
Parts:
- removed the SW_ACTION at (77.1, 61.1)
- removed the SW_DOWN at (19.7, 77.8)
- removed the SW_LEFT at (10.7, 68.8)
- removed the SW_MENU at (39.6, 85.4)
- removed the SW_RESET at (56.5, 81.6)
- removed the SW_RIGHT at (28.7, 68.8)
- removed the SW_UNDO at (60.4, 65.8)
- removed the SW_UP at (19.7, 59.8)
- added SW_ACTION: SW_SPST_EVQP2_MiddlePushTravel_H2.5mm, SW_SPST_EVQP2_MiddlePushTravel_H2.5mm, F.Cu at (77.1, 61.1)
- added SW_DOWN: SW_SPST_EVQP2_MiddlePushTravel_H2.5mm, SW_SPST_EVQP2_MiddlePushTravel_H2.5mm, F.Cu at (19.7, 77.8)
- added SW_LEFT: SW_SPST_EVQP2_MiddlePushTravel_H2.5mm, SW_SPST_EVQP2_MiddlePushTravel_H2.5mm, F.Cu at (10.7, 68.8)
- added SW_MENU: SW_SPST_EVQP2_MiddlePushTravel_H2.5mm, SW_SPST_EVQP2_MiddlePushTravel_H2.5mm, F.Cu at (39.6, 85.4)
- added SW_RESET: SW_SPST_EVQP2_MiddlePushTravel_H2.5mm, SW_SPST_EVQP2_MiddlePushTravel_H2.5mm, F.Cu at (56.5, 81.6)
- added SW_RIGHT: SW_SPST_EVQP2_MiddlePushTravel_H2.5mm, SW_SPST_EVQP2_MiddlePushTravel_H2.5mm, F.Cu at (28.7, 68.8)
- added SW_UNDO: SW_SPST_EVQP2_MiddlePushTravel_H2.5mm, SW_SPST_EVQP2_MiddlePushTravel_H2.5mm, F.Cu at (60.4, 65.8)
- added SW_UP: SW_SPST_EVQP2_MiddlePushTravel_H2.5mm, SW_SPST_EVQP2_MiddlePushTravel_H2.5mm, F.Cu at (19.7, 59.8)
Connections:
- J_BAT_IN pad 1: (no net) -> BAT_P
- J_BAT_IN pad 2: (no net) -> GND
- J_BAT_OUT pad 1: (no net) -> BAT_SW
- J_BAT_OUT pad 2: (no net) -> GND
- J_EXP pad 1: (no net) -> INT
- J_I2C pad 1: (no net) -> +3V3
- J_I2C pad 2: (no net) -> GND
- J_I2C pad 3: (no net) -> SCL
- J_I2C pad 4: (no net) -> SDA
- SW_MUTE pad : (no net) -> GND
- SW_MUTE pad 1: (no net) -> SIG_MUTE
- SW_MUTE pad 2: (no net) -> GND
- SW_MUTE pad 3: (no net) -> GND
- SW_PWR pad 1: (no net) -> BAT_SW
- SW_PWR pad 2: (no net) -> BAT_P
- U1 pad 1: (no net) -> SIG_UP
- U1 pad 10: (no net) -> GND
- U1 pad 12: (no net) -> SCL
- U1 pad 13: (no net) -> SDA
- U1 pad 15: (no net) -> GND
- U1 pad 16: (no net) -> GND
- U1 pad 17: (no net) -> GND
- U1 pad 18: (no net) -> +3V3
- U1 pad 20: (no net) -> INT
- U1 pad 21: (no net) -> SIG_DOWN
- U1 pad 22: (no net) -> SIG_RESET
- U1 pad 23: (no net) -> SIG_MENU
- U1 pad 24: (no net) -> SIG_LEFT
- U1 pad 25: (no net) -> SIG_RIGHT
- U1 pad 26: (no net) -> SIG_UNDO
- U1 pad 27: (no net) -> SIG_MUTE
- U1 pad 28: (no net) -> SIG_ACTION
- U1 pad 9: (no net) -> +3V3
Routing:
- net GND: track 0.00 -> 89.3 mm
- net BAT_SW: track 0.00 -> 65.5 mm, vias 0 -> 2
- net SDA: track 0.00 -> 53.0 mm, vias 0 -> 2
- net BAT_P: track 0.00 -> 49.0 mm
- net +3V3: track 0.00 -> 48.8 mm, vias 0 -> 4
- net SIG_LEFT: track 0.00 -> 42.3 mm, vias 0 -> 2
- net SCL: track 0.00 -> 38.0 mm
- net SIG_DOWN: track 0.00 -> 36.5 mm, vias 0 -> 2
- net INT: track 0.00 -> 33.6 mm, vias 0 -> 2
- net SIG_ACTION: track 0.00 -> 33.2 mm
- net SIG_UP: track 0.00 -> 30.9 mm
- net SIG_MUTE: track 0.00 -> 30.0 mm
- net SIG_MENU: track 0.00 -> 25.7 mm
- net SIG_RIGHT: track 0.00 -> 24.3 mm, vias 0 -> 2
- net SIG_RESET: track 0.00 -> 16.5 mm
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- added copper zone on B.Cu, net GND
- added copper zone on F.Cu, net GND

Commit message: work on pocket card pcbs
Parts:
- removed the SW_ACTION at (77.1, 61.1)
- removed the SW_DOWN at (19.7, 77.8)
- removed the SW_LEFT at (10.7, 68.8)
- removed the SW_RESET at (56.5, 81.6)
- removed the SW_RIGHT at (28.7, 68.8)
- removed the SW_UNDO at (60.4, 65.8)
- removed the SW_UP at (19.7, 59.8)
- added SW_ACTION: SW_SPST_EVQP0, SW_SPST_EVQP0, F.Cu at (77.1, 61.1)
- added SW_DOWN: SW_SPST_EVQP0, SW_SPST_EVQP0, F.Cu at (19.7, 77.8)
- added SW_LEFT: SW_SPST_EVQP0, SW_SPST_EVQP0, F.Cu at (10.7, 68.8)
- added SW_RESET: SW_SPST_EVQP0, SW_SPST_EVQP0, F.Cu at (56.5, 81.6)
- added SW_RIGHT: SW_SPST_EVQP0, SW_SPST_EVQP0, F.Cu at (28.7, 68.8)
- added SW_UNDO: SW_SPST_EVQP0, SW_SPST_EVQP0, F.Cu at (60.4, 65.8)
- added SW_UP: SW_SPST_EVQP0, SW_SPST_EVQP0, F.Cu at (19.7, 59.8)
Routing:
- net SDA: track 53.0 -> 41.2 mm, vias 2 -> 0
- net +3V3: track 48.8 -> 57.4 mm, vias 4 -> 2
- net SIG_LEFT: track 42.3 -> 50.5 mm
- net GND: track 89.3 -> 81.1 mm
- net SIG_RESET: track 16.5 -> 24.2 mm, vias 0 -> 2
- net INT: track 33.6 -> 26.1 mm, vias 2 -> 0
- net SIG_RIGHT: track 24.3 -> 30.2 mm, vias 2 -> 3
- net SIG_UP: track 30.9 -> 26.0 mm
- net SIG_UNDO: track 13.9 -> 18.7 mm, vias 0 -> 2
- net BAT_SW: track 65.5 -> 60.9 mm
- net SIG_MUTE: track 30.0 -> 25.6 mm
- net SCL: track 38.0 -> 40.9 mm
- net SIG_MENU: track 25.7 -> 22.9 mm
- net SIG_ACTION: track 33.2 -> 32.3 mm
- net SIG_DOWN: track 36.5 -> 35.7 mm
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