File: hardware/pocket_card/case/out/pcb/pocket_card_controller.kicad_pcb (KiCad board)
At the start: 2 copper layers, 80.5 x 37 mm, 19 parts, among them U1 SOIC-28W_7.5x17.9mm_P1.27mm

Commit message: Place SKQG on front and module JSTs on PCB back.
All eight sites use SW_SPST_SKQG_WithStem on F.Cu; GH connectors flip to B.Cu
in the right-rear pocket at courtyard-clear pitches. pcb.py emits boards
headless from .kicad_mod (wx/pcbnew hangs in this environment). Pocket and
SKQG keepout checks gate the anchors.

Co-authored-by: Cursor <cursoragent@cursor.com>
Parts:
- removed the SW_ACTION at (77.1, 61.1)
- removed the SW_DOWN at (19.7, 77.8)
- removed the SW_LEFT at (10.7, 68.8)
- removed the SW_MENU at (39.6, 85.4)
- removed the SW_RESET at (56.5, 81.6)
- removed the SW_RIGHT at (28.7, 68.8)
- removed the SW_UNDO at (60.4, 65.8)
- removed the SW_UP at (19.7, 59.8)
- added SW_ACTION: SW_SPST_SKQG_WithStem, SW_SPST_SKQG_WithStem, F.Cu at (77.1, 61.1)
- added SW_DOWN: SW_SPST_SKQG_WithStem, SW_SPST_SKQG_WithStem, F.Cu at (19.7, 77.8)
- added SW_LEFT: SW_SPST_SKQG_WithStem, SW_SPST_SKQG_WithStem, F.Cu at (10.7, 68.8)
- added SW_MENU: SW_SPST_SKQG_WithStem, SW_SPST_SKQG_WithStem, F.Cu at (39.6, 85.4)
- added SW_RESET: SW_SPST_SKQG_WithStem, SW_SPST_SKQG_WithStem, F.Cu at (56.5, 81.6)
- added SW_RIGHT: SW_SPST_SKQG_WithStem, SW_SPST_SKQG_WithStem, F.Cu at (28.7, 68.8)
- added SW_UNDO: SW_SPST_SKQG_WithStem, SW_SPST_SKQG_WithStem, F.Cu at (60.4, 65.8)
- added SW_UP: SW_SPST_SKQG_WithStem, SW_SPST_SKQG_WithStem, F.Cu at (19.7, 59.8)
- J_BAT_IN, J_BAT_OUT, J_EXP, J_I2C: moved to B.Cu
- moved J_I2C 62.1 mm to (74.0, 58.0)
- moved J_EXP 41.4 mm to (74.0, 65.0)
- moved J_BAT_IN 33.0 mm to (74.0, 72.0)
- moved J_BAT_OUT 30.4 mm to (74.0, 79.0)
Connections:
- J_BAT_IN pad 1: BAT_P -> (no net)
- J_BAT_IN pad 2: GND -> (no net)
- J_BAT_OUT pad 1: BAT_SW -> (no net)
- J_BAT_OUT pad 2: GND -> (no net)
- J_EXP pad 1: INT -> (no net)
- J_I2C pad 1: +3V3 -> (no net)
- J_I2C pad 2: GND -> (no net)
- J_I2C pad 3: SCL -> (no net)
- J_I2C pad 4: SDA -> (no net)
- SW_MUTE pad : GND -> (no net)
- SW_MUTE pad 1: SIG_MUTE -> (no net)
- SW_MUTE pad 2: GND -> (no net)
- SW_MUTE pad 3: GND -> (no net)
- SW_PWR pad 1: BAT_SW -> (no net)
- SW_PWR pad 2: BAT_P -> (no net)
- U1 pad 1: SIG_UP -> (no net)
- U1 pad 10: GND -> (no net)
- U1 pad 12: SCL -> (no net)
- U1 pad 13: SDA -> (no net)
- U1 pad 15: GND -> (no net)
- U1 pad 16: GND -> (no net)
- U1 pad 17: GND -> (no net)
- U1 pad 18: +3V3 -> (no net)
- U1 pad 20: INT -> (no net)
- U1 pad 21: SIG_DOWN -> (no net)
- U1 pad 22: SIG_RESET -> (no net)
- U1 pad 23: SIG_MENU -> (no net)
- U1 pad 24: SIG_LEFT -> (no net)
- U1 pad 25: SIG_RIGHT -> (no net)
- U1 pad 26: SIG_UNDO -> (no net)
- U1 pad 27: SIG_MUTE -> (no net)
- U1 pad 28: SIG_ACTION -> (no net)
- U1 pad 9: +3V3 -> (no net)
Routing:
- net GND: track 81.1 -> 0.00 mm
- net BAT_SW: track 60.9 -> 0.00 mm, vias 2 -> 0
- net +3V3: track 57.4 -> 0.00 mm, vias 2 -> 0
- net SIG_LEFT: track 50.5 -> 0.00 mm, vias 2 -> 0
- net BAT_P: track 48.9 -> 0.00 mm, vias 2 -> 0
- net SDA: track 41.2 -> 0.00 mm
- net SCL: track 40.9 -> 0.00 mm
- net SIG_DOWN: track 35.7 -> 0.00 mm, vias 2 -> 0
- net SIG_ACTION: track 32.3 -> 0.00 mm
- net SIG_RIGHT: track 30.2 -> 0.00 mm, vias 3 -> 0
- net INT: track 26.1 -> 0.00 mm
- net SIG_UP: track 26.0 -> 0.00 mm
- net SIG_MUTE: track 25.6 -> 0.00 mm
- net SIG_RESET: track 24.2 -> 0.00 mm, vias 2 -> 0
- net SIG_MENU: track 22.9 -> 0.00 mm
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- removed copper zone on B.Cu, net GND
- removed copper zone on F.Cu, net GND

Commit message: Route Pocket Card controller after SKQG and rear JST move.
Headless freerouting rebuild: dual-layer GND pour with stitch vias, JST MP
pads on GND, slides clear of the board edge and Reset courtyard. pcb_reroute
no longer strips SKQG footprint keepouts. DRC: 0 errors, 0 unconnected.

Co-authored-by: Cursor <cursoragent@cursor.com>
Parts:
- moved SW_MUTE 10.2 mm to (70.0, 86.5)
- moved SW_PWR 2.00 mm to (20.0, 86.5)
Connections:
- J_BAT_IN pad 1: (no net) -> BAT_P
- J_BAT_IN pad 2: (no net) -> GND
- J_BAT_IN pad MP: (no net) -> GND
- J_BAT_OUT pad 1: (no net) -> BAT_SW
- J_BAT_OUT pad 2: (no net) -> GND
- J_BAT_OUT pad MP: (no net) -> GND
- J_EXP pad 1: (no net) -> INT
- J_EXP pad MP: (no net) -> GND
- J_I2C pad 1: (no net) -> +3V3
- J_I2C pad 2: (no net) -> GND
- J_I2C pad 3: (no net) -> SCL
- J_I2C pad 4: (no net) -> SDA
- J_I2C pad MP: (no net) -> GND
- SW_ACTION pad 1: (no net) -> SIG_ACTION
- SW_ACTION pad 2: (no net) -> GND
- SW_DOWN pad 1: (no net) -> SIG_DOWN
- SW_DOWN pad 2: (no net) -> GND
- SW_LEFT pad 1: (no net) -> SIG_LEFT
- SW_LEFT pad 2: (no net) -> GND
- SW_MENU pad 1: (no net) -> SIG_MENU
- SW_MENU pad 2: (no net) -> GND
- SW_MUTE pad : (no net) -> GND
- SW_MUTE pad 1: (no net) -> SIG_MUTE
- SW_MUTE pad 2: (no net) -> GND
- SW_MUTE pad 3: (no net) -> GND
- SW_PWR pad 1: (no net) -> BAT_SW
- SW_PWR pad 2: (no net) -> BAT_P
- SW_RESET pad 1: (no net) -> SIG_RESET
- SW_RESET pad 2: (no net) -> GND
- SW_RIGHT pad 1: (no net) -> SIG_RIGHT
- SW_RIGHT pad 2: (no net) -> GND
- SW_UNDO pad 1: (no net) -> SIG_UNDO
- SW_UNDO pad 2: (no net) -> GND
- SW_UP pad 1: (no net) -> SIG_UP
- SW_UP pad 2: (no net) -> GND
- U1 pad 1: (no net) -> SIG_UP
- U1 pad 10: (no net) -> GND
- U1 pad 12: (no net) -> SCL
- U1 pad 13: (no net) -> SDA
- U1 pad 15: (no net) -> GND
- U1 pad 16: (no net) -> GND
- U1 pad 17: (no net) -> GND
- U1 pad 18: (no net) -> +3V3
- U1 pad 20: (no net) -> INT
- U1 pad 21: (no net) -> SIG_DOWN
- U1 pad 22: (no net) -> SIG_RESET
- U1 pad 23: (no net) -> SIG_MENU
- U1 pad 24: (no net) -> SIG_LEFT
- U1 pad 25: (no net) -> SIG_RIGHT
- U1 pad 26: (no net) -> SIG_UNDO
- U1 pad 27: (no net) -> SIG_MUTE
- U1 pad 28: (no net) -> SIG_ACTION
- U1 pad 9: (no net) -> +3V3
Routing:
- net GND: track 0.00 -> 233.9 mm, vias 0 -> 9
- net BAT_P: track 0.00 -> 61.9 mm, vias 0 -> 1
- net BAT_SW: track 0.00 -> 59.4 mm, vias 0 -> 1
- net +3V3: track 0.00 -> 48.4 mm, vias 0 -> 2
- net SDA: track 0.00 -> 46.4 mm, vias 0 -> 1
- net SIG_DOWN: track 0.00 -> 45.0 mm
- net SIG_LEFT: track 0.00 -> 44.2 mm, vias 0 -> 2
- net SCL: track 0.00 -> 43.3 mm, vias 0 -> 1
- net SIG_ACTION: track 0.00 -> 32.4 mm
- net SIG_MUTE: track 0.00 -> 30.7 mm
- net INT: track 0.00 -> 29.7 mm, vias 0 -> 1
- net SIG_UP: track 0.00 -> 26.2 mm, vias 0 -> 1
- net SIG_RIGHT: track 0.00 -> 25.8 mm
- net SIG_MENU: track 0.00 -> 23.4 mm
- net SIG_RESET: track 0.00 -> 19.6 mm
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- added copper zone on B.Cu, net GND
- added copper zone on F.Cu, net GND

Commit message: Fix slide openings and give GH plugs room toward the module.
Order STLs were stale. Shell power/mute cuts now track switch XY with a
PCM12-sized aperture (was a 5 mm letterbox on a fixed Y). JSTs move to a
2×2 B.Cu grid at rot=0 so mouths clear each other and face the module.

Co-authored-by: Cursor <cursoragent@cursor.com>
Parts:
- moved J_I2C 12.1 mm to (63.0, 63.0), turned to 0 degrees
- moved J_BAT_IN 11.7 mm to (63.0, 76.0), turned to 0 degrees
- moved J_BAT_OUT 5.00 mm to (78.0, 76.0), turned to 0 degrees
- moved J_EXP 4.47 mm to (78.0, 63.0), turned to 0 degrees
Routing:
- net GND: track 233.9 -> 262.1 mm
- net BAT_P: track 61.9 -> 46.8 mm
- net +3V3: track 48.4 -> 33.6 mm, vias 2 -> 1
- net SCL: track 43.3 -> 30.8 mm
- net SDA: track 46.4 -> 38.7 mm
- net INT: track 29.7 -> 36.0 mm
- net BAT_SW: track 59.4 -> 65.7 mm
- net SIG_MENU: track 23.4 -> 28.5 mm
- net SIG_UNDO: track 14.8 -> 17.8 mm
- net SIG_DOWN: track 45.0 -> 42.3 mm, vias 0 -> 3
- net SIG_RESET: track 19.6 -> 17.0 mm
- net SIG_MUTE: track 30.7 -> 28.5 mm
- net SIG_LEFT: track 44.2 -> 45.8 mm
- net SIG_RIGHT: track 25.8 -> 24.3 mm
- net SIG_UP: vias 1 -> 0

Commit message: Swap power/mute to JS102011 and notch the PCB south edge.
Co-authored-by: Cursor <cursoragent@cursor.com>
Parts:
- removed the SW_MUTE at (70.0, 86.5)
- removed the SW_PWR at (20.0, 86.5)
- added SW_MUTE: SW_SPDT_CK_JS102011SAQN, SW_SPDT_CK_JS102011SAQN, F.Cu at (70.0, 88.0)
- added SW_PWR: SW_SPDT_CK_JS102011SAQN, SW_SPDT_CK_JS102011SAQN, F.Cu at (20.0, 88.0)
Connections:
- J_BAT_IN pad 1: BAT_P -> (no net)
- J_BAT_IN pad 2: GND -> (no net)
- J_BAT_IN pad MP: GND -> (no net)
- J_BAT_OUT pad 1: BAT_SW -> (no net)
- J_BAT_OUT pad 2: GND -> (no net)
- J_BAT_OUT pad MP: GND -> (no net)
- J_EXP pad 1: INT -> (no net)
- J_EXP pad MP: GND -> (no net)
- J_I2C pad 1: +3V3 -> (no net)
- J_I2C pad 2: GND -> (no net)
- J_I2C pad 3: SCL -> (no net)
- J_I2C pad 4: SDA -> (no net)
- J_I2C pad MP: GND -> (no net)
- SW_ACTION pad 1: SIG_ACTION -> (no net)
- SW_ACTION pad 2: GND -> (no net)
- SW_DOWN pad 1: SIG_DOWN -> (no net)
- SW_DOWN pad 2: GND -> (no net)
- SW_LEFT pad 1: SIG_LEFT -> (no net)
- SW_LEFT pad 2: GND -> (no net)
- SW_MENU pad 1: SIG_MENU -> (no net)
- SW_MENU pad 2: GND -> (no net)
- SW_RESET pad 1: SIG_RESET -> (no net)
- SW_RESET pad 2: GND -> (no net)
- SW_RIGHT pad 1: SIG_RIGHT -> (no net)
- SW_RIGHT pad 2: GND -> (no net)
- SW_UNDO pad 1: SIG_UNDO -> (no net)
- SW_UNDO pad 2: GND -> (no net)
- SW_UP pad 1: SIG_UP -> (no net)
- SW_UP pad 2: GND -> (no net)
- U1 pad 1: SIG_UP -> (no net)
- U1 pad 10: GND -> (no net)
- U1 pad 12: SCL -> (no net)
- U1 pad 13: SDA -> (no net)
- U1 pad 15: GND -> (no net)
- U1 pad 16: GND -> (no net)
- U1 pad 17: GND -> (no net)
- U1 pad 18: +3V3 -> (no net)
- U1 pad 20: INT -> (no net)
- U1 pad 21: SIG_DOWN -> (no net)
- U1 pad 22: SIG_RESET -> (no net)
- U1 pad 23: SIG_MENU -> (no net)
- U1 pad 24: SIG_LEFT -> (no net)
- U1 pad 25: SIG_RIGHT -> (no net)
- U1 pad 26: SIG_UNDO -> (no net)
- U1 pad 27: SIG_MUTE -> (no net)
- U1 pad 28: SIG_ACTION -> (no net)
- U1 pad 9: +3V3 -> (no net)
Routing:
- net GND: track 262.1 -> 0.00 mm, vias 9 -> 0
- net BAT_SW: track 65.7 -> 0.00 mm, vias 1 -> 0
- net BAT_P: track 46.8 -> 0.00 mm, vias 1 -> 0
- net SIG_LEFT: track 45.8 -> 0.00 mm, vias 2 -> 0
- net SIG_DOWN: track 42.3 -> 0.00 mm, vias 3 -> 0
- net SDA: track 38.7 -> 0.00 mm, vias 1 -> 0
- net INT: track 36.0 -> 0.00 mm, vias 1 -> 0
- net +3V3: track 33.6 -> 0.00 mm, vias 1 -> 0
- net SIG_ACTION: track 32.4 -> 0.00 mm
- net SCL: track 30.8 -> 0.00 mm, vias 1 -> 0
- net SIG_MUTE: track 28.5 -> 0.00 mm
- net SIG_MENU: track 28.5 -> 0.00 mm
- net SIG_UP: track 26.2 -> 0.00 mm
- net SIG_RIGHT: track 24.3 -> 0.00 mm
- net SIG_UNDO: track 17.8 -> 0.00 mm
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- removed copper zone on B.Cu, net GND
- removed copper zone on F.Cu, net GND
Other:
- outline, holes or cut-outs redrawn
