File: hardware/pocket_card/case/out/pcb/pocket_card_controller.kicad_pcb (KiCad board)
At the start: 2 copper layers, 80.5 x 37 mm, 19 parts, among them U1 SOIC-28W_7.5x17.9mm_P1.27mm

Commit message: eda case firstprototype
Parts:
- removed the SW_MUTE at (74.0, 88.0)
- removed the SW_PWR at (20.0, 88.0)
- added SW_MUTE: SW_SPDT_PCM12, SW_SPDT_PCM12, F.Cu at (58.0, 87.7)
- added SW_PWR: SW_SPDT_PCM12, SW_SPDT_PCM12, F.Cu at (20.0, 87.7)
- moved SW_RESET 1.60 mm to (56.5, 80.0)
Routing:
- net GND: track 248.8 -> 263.2 mm, vias 10 -> 8
- net SDA: track 32.0 -> 45.3 mm
- net INT: track 42.2 -> 33.8 mm
- net SIG_MUTE: track 40.7 -> 33.4 mm
- net SIG_RESET: track 23.0 -> 16.1 mm, vias 0 -> 1
- net BAT_P: track 53.5 -> 47.2 mm
- net SIG_ACTION: track 38.6 -> 32.4 mm
- net SCL: track 45.2 -> 39.6 mm
- net SIG_MENU: track 26.0 -> 28.5 mm
- net BAT_SW: track 67.2 -> 69.5 mm
- net SIG_LEFT: track 52.8 -> 50.9 mm
- net +3V3: track 33.3 -> 34.5 mm
- net SIG_UNDO: track 14.8 -> 15.5 mm, vias 0 -> 2
- net SIG_DOWN: track 37.4 -> 37.7 mm, vias 0 -> 2
Other:
- outline, holes or cut-outs redrawn
