File: hardware/pocket_card/case/out/pcb/pocket_card_controller.kicad_sch (KiCad schematic)
At the start: 17 parts, among them U1 MCP23017-E/SO

Commit message: docs: audit pocket card controller circuit
Changed lines of the file:
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@@
       (path "/2e13cb0c-6647-4fc9-a0db-5ca9b27d688a" (reference "H2") (unit 1))))
   )
+  (symbol (lib_id "PocketCard:PWR_FLAG") (at 60 27.5 0) (unit 1)
+    (exclude_from_sim yes) (in_bom no) (on_board no) (dnp no)
+    (property "Reference" "#FLG01" (at 60 23.69 0)
+      (effects (font (size 1.27 1.27)) hide))
+    (property "Value" "PWR_FLAG" (at 60 31.31 0)
+      (effects (font (size 1.27 1.27))))
+    (property "Footprint" "" (at 60 27.5 0)
+      (effects (font (size 1.27 1.27)) hide))
+    (property "Datasheet" "~" (at 60 27.5 0)
+      (effects (font (size 1.27 1.27)) hide))
+    (pin "1")
+    (instances (project "pocket_card_controller"
+      (path "/2e13cb0c-6647-4fc9-a0db-5ca9b27d688a" (reference "#FLG01") (unit 1))))
+  )
+  (symbol (lib_id "PocketCard:PWR_FLAG") (at 90 27.5 0) (unit 1)
+    (exclude_from_sim yes) (in_bom no) (on_board no) (dnp no)
+    (property "Reference" "#FLG02" (at 90 23.69 0)
+      (effects (font (size 1.27 1.27)) hide))
+    (property "Value" "PWR_FLAG" (at 90 31.31 0)
+      (effects (font (size 1.27 1.27))))
+    (property "Footprint" "" (at 90 27.5 0)
+      (effects (font (size 1.27 1.27)) hide))
+    (property "Datasheet" "~" (at 90 27.5 0)
+      (effects (font (size 1.27 1.27)) hide))
+    (pin "1")
+    (instances (project "pocket_card_controller"
+      (path "/2e13cb0c-6647-4fc9-a0db-5ca9b27d688a" (reference "#FLG02") (unit 1))))
+  )
   (wire
     (pts (xy 92.3 66.19) (xy 87.22 66.19))
@@
     (effects (font (size 1.27 1.27)) (justify left))
   )
+  (wire
+    (pts (xy 60 24.96) (xy 60 19.88))
+    (stroke (width 0) (type default))
+  )
+  (label "+3V3" (at 60 19.88 0) (fields_autoplaced)
+    (effects (font (size 1.27 1.27)) (justify left))
+  )
+  (wire
+    (pts (xy 90 24.96) (xy 90 19.88))
+    (stroke (width 0) (type default))
+  )
+  (label "GND" (at 90 19.88 0) (fields_autoplaced)
+    (effects (font (size 1.27 1.27)) (justify left))
+  )
