File: hardware/pocket_card/case/out/pcb/pocket_card_controller.kicad_sch (KiCad schematic)
At the start: 17 parts, among them U1 MCP23017-E/SO

Commit message: fix: fully annotate Pocket Card schematic
Parts:
- J_EXP1: renamed from J_EXP; NC Audit 2 NC J_EXP.2 -> NC J_EXP1.2; NC Audit 3 NC J_EXP.3 -> NC J_EXP1.3; NC Audit 4 NC J_EXP.4 -> NC J_EXP1.4
- SW_PWR1: renamed from SW_PWR; NC Audit 3 NC SW_PWR.3 -> NC SW_PWR1.3
- renumbered J_BAT_IN to J_BAT_IN1, J_BAT_OUT to J_BAT_OUT1, J_I2C to J_I2C1, SW_ACTION to SW_ACTION1, SW_DOWN to SW_DOWN1, SW_LEFT to SW_LEFT1, SW_MENU to SW_MENU1, SW_MUTE to SW_MUTE1, SW_RESET to SW_RESET1, SW_RIGHT to SW_RIGHT1, SW_UNDO to SW_UNDO1, SW_UP to SW_UP1
Changed lines of the file:
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@@
   (symbol (lib_id "PocketCard:Tact") (at 185 30 0) (unit 1)
     (exclude_from_sim no) (in_bom yes) (on_board yes) (dnp no)
-    (property "Reference" "SW_UP" (at 185 24.92 0)
+    (property "Reference" "SW_UP1" (at 185 24.92 0)
       (effects (font (size 1.27 1.27))))
     (property "Value" "SKQGABE010" (at 185 35.08 0)
@@
     (pin "2")
     (instances (project "pocket_card_controller"
-      (path "/2e13cb0c-6647-4fc9-a0db-5ca9b27d688a" (reference "SW_UP") (unit 1))))
+      (path "/2e13cb0c-6647-4fc9-a0db-5ca9b27d688a" (reference "SW_UP1") (unit 1))))
   )
   (symbol (lib_id "PocketCard:Tact") (at 185 50 0) (unit 1)
     (exclude_from_sim no) (in_bom yes) (on_board yes) (dnp no)
-    (property "Reference" "SW_DOWN" (at 185 44.92 0)
+    (property "Reference" "SW_DOWN1" (at 185 44.92 0)
       (effects (font (size 1.27 1.27))))
     (property "Value" "SKQGABE010" (at 185 55.08 0)
@@
     (pin "2")
     (instances (project "pocket_card_controller"
-      (path "/2e13cb0c-6647-4fc9-a0db-5ca9b27d688a" (reference "SW_DOWN") (unit 1))))
+      (path "/2e13cb0c-6647-4fc9-a0db-5ca9b27d688a" (reference "SW_DOWN1") (unit 1))))
   )
   (symbol (lib_id "PocketCard:Tact") (at 185 70 0) (unit 1)
     (exclude_from_sim no) (in_bom yes) (on_board yes) (dnp no)
-    (property "Reference" "SW_LEFT" (at 185 64.92 0)
+    (property "Reference" "SW_LEFT1" (at 185 64.92 0)
       (effects (font (size 1.27 1.27))))
     (property "Value" "SKQGABE010" (at 185 75.08 0)
@@
     (pin "2")
     (instances (project "pocket_card_controller"
-      (path "/2e13cb0c-6647-4fc9-a0db-5ca9b27d688a" (reference "SW_LEFT") (unit 1))))
+      (path "/2e13cb0c-6647-4fc9-a0db-5ca9b27d688a" (reference "SW_LEFT1") (unit 1))))
   )
   (symbol (lib_id "PocketCard:Tact") (at 185 90 0) (unit 1)
     (exclude_from_sim no) (in_bom yes) (on_board yes) (dnp no)
-    (property "Reference" "SW_RIGHT" (at 185 84.92 0)
+    (property "Reference" "SW_RIGHT1" (at 185 84.92 0)
       (effects (font (size 1.27 1.27))))
     (property "Value" "SKQGABE010" (at 185 95.08 0)
@@
     (pin "2")
     (instances (project "pocket_card_controller"
-      (path "/2e13cb0c-6647-4fc9-a0db-5ca9b27d688a" (reference "SW_RIGHT") (unit 1))))
+      (path "/2e13cb0c-6647-4fc9-a0db-5ca9b27d688a" (reference "SW_RIGHT1") (unit 1))))
   )
   (symbol (lib_id "PocketCard:Tact") (at 235 30 0) (unit 1)
     (exclude_from_sim no) (in_bom yes) (on_board yes) (dnp no)
-    (property "Reference" "SW_UNDO" (at 235 24.92 0)
+    (property "Reference" "SW_UNDO1" (at 235 24.92 0)
       (effects (font (size 1.27 1.27))))
     (property "Value" "SKQGABE010" (at 235 35.08 0)
@@
     (pin "2")
     (instances (project "pocket_card_controller"
-      (path "/2e13cb0c-6647-4fc9-a0db-5ca9b27d688a" (reference "SW_UNDO") (unit 1))))
+      (path "/2e13cb0c-6647-4fc9-a0db-5ca9b27d688a" (reference "SW_UNDO1") (unit 1))))
   )
   (symbol (lib_id "PocketCard:Tact") (at 235 50 0) (unit 1)
     (exclude_from_sim no) (in_bom yes) (on_board yes) (dnp no)
-    (property "Reference" "SW_ACTION" (at 235 44.92 0)
+    (property "Reference" "SW_ACTION1" (at 235 44.92 0)
       (effects (font (size 1.27 1.27))))
     (property "Value" "SKQGABE010" (at 235 55.08 0)
@@
     (pin "2")
     (instances (project "pocket_card_controller"
-      (path "/2e13cb0c-6647-4fc9-a0db-5ca9b27d688a" (reference "SW_ACTION") (unit 1))))
+      (path "/2e13cb0c-6647-4fc9-a0db-5ca9b27d688a" (reference "SW_ACTION1") (unit 1))))
   )
   (symbol (lib_id "PocketCard:Tact") (at 235 70 0) (unit 1)
     (exclude_from_sim no) (in_bom yes) (on_board yes) (dnp no)
-    (property "Reference" "SW_RESET" (at 235 64.92 0)
+    (property "Reference" "SW_RESET1" (at 235 64.92 0)
       (effects (font (size 1.27 1.27))))
     (property "Value" "SKQGABE010" (at 235 75.08 0)
@@
     (pin "2")
     (instances (project "pocket_card_controller"
-      (path "/2e13cb0c-6647-4fc9-a0db-5ca9b27d688a" (reference "SW_RESET") (unit 1))))
+      (path "/2e13cb0c-6647-4fc9-a0db-5ca9b27d688a" (reference "SW_RESET1") (unit 1))))
   )
   (symbol (lib_id "PocketCard:Tact") (at 235 90 0) (unit 1)
     (exclude_from_sim no) (in_bom yes) (on_board yes) (dnp no)
-    (property "Reference" "SW_MENU" (at 235 84.92 0)
+    (property "Reference" "SW_MENU1" (at 235 84.92 0)
       (effects (font (size 1.27 1.27))))
     (property "Value" "SKQGABE010" (at 235 95.08 0)
@@
     (pin "2")
     (instances (project "pocket_card_controller"
-      (path "/2e13cb0c-6647-4fc9-a0db-5ca9b27d688a" (reference "SW_MENU") (unit 1))))
+      (path "/2e13cb0c-6647-4fc9-a0db-5ca9b27d688a" (reference "SW_MENU1") (unit 1))))
   )
   (symbol (lib_id "PocketCard:SlideSPDT") (at 105 130 0) (unit 1)
     (exclude_from_sim no) (in_bom yes) (on_board yes) (dnp no)
-    (property "Reference" "SW_PWR" (at 105 123.65 0)
+    (property "Reference" "SW_PWR1" (at 105 123.65 0)
       (effects (font (size 1.27 1.27))))
     (property "Value" "PCM12SMTR" (at 105 136.35 0)
@@
     (property "Datasheet" "~" (at 105 130 0)
       (effects (font (size 1.27 1.27)) hide))
-    (property "NC Audit 3" "NC SW_PWR.3" (at 105 130 0)
-      (effects (font (size 1.27 1.27)) hide))
-    (pin "1")
-    (pin "2")
-    (pin "3")
-    (instances (project "pocket_card_controller"
-      (path "/2e13cb0c-6647-4fc9-a0db-5ca9b27d688a" (reference "SW_PWR") (unit 1))))
+    (property "NC Audit 3" "NC SW_PWR1.3" (at 105 130 0)
+      (effects (font (size 1.27 1.27)) hide))
+    (pin "1")
+    (pin "2")
+    (pin "3")
+    (instances (project "pocket_card_controller"
+      (path "/2e13cb0c-6647-4fc9-a0db-5ca9b27d688a" (reference "SW_PWR1") (unit 1))))
   )
   (symbol (lib_id "PocketCard:SlideSPDT") (at 235 115 0) (unit 1)
     (exclude_from_sim no) (in_bom yes) (on_board yes) (dnp no)
-    (property "Reference" "SW_MUTE" (at 235 108.65 0)
+    (property "Reference" "SW_MUTE1" (at 235 108.65 0)
       (effects (font (size 1.27 1.27))))
     (property "Value" "PCM12SMTR" (at 235 121.35 0)
@@
     (pin "3")
     (instances (project "pocket_card_controller"
-      (path "/2e13cb0c-6647-4fc9-a0db-5ca9b27d688a" (reference "SW_MUTE") (unit 1))))
+      (path "/2e13cb0c-6647-4fc9-a0db-5ca9b27d688a" (reference "SW_MUTE1") (unit 1))))
   )
   (symbol (lib_id "PocketCard:JST4") (at 35 35 0) (unit 1)
     (exclude_from_sim no) (in_bom yes) (on_board yes) (dnp no)
-    (property "Reference" "J_I2C" (at 26.11 28.65 0)
+    (property "Reference" "J_I2C1" (at 26.11 28.65 0)
       (effects (font (size 1.27 1.27))))
     (property "Value" "WAFER-GH1.25-4PWB" (at 35 45.16 0)
@@
     (pin "MP")
     (instances (project "pocket_card_controller"
-      (path "/2e13cb0c-6647-4fc9-a0db-5ca9b27d688a" (reference "J_I2C") (unit 1))))
+      (path "/2e13cb0c-6647-4fc9-a0db-5ca9b27d688a" (reference "J_I2C1") (unit 1))))
   )
   (symbol (lib_id "PocketCard:JST4") (at 35 75 0) (unit 1)
     (exclude_from_sim no) (in_bom yes) (on_board yes) (dnp no)
-    (property "Reference" "J_EXP" (at 26.11 68.65 0)
+    (property "Reference" "J_EXP1" (at 26.11 68.65 0)
       (effects (font (size 1.27 1.27))))
     (property "Value" "WAFER-GH1.25-4PWB" (at 35 85.16 0)
@@
     (property "Datasheet" "~" (at 35 75 0)
       (effects (font (size 1.27 1.27)) hide))
-    (property "NC Audit 2" "NC J_EXP.2" (at 35 75 0)
-      (effects (font (size 1.27 1.27)) hide))
-    (property "NC Audit 3" "NC J_EXP.3" (at 35 75 0)
-      (effects (font (size 1.27 1.27)) hide))
-    (property "NC Audit 4" "NC J_EXP.4" (at 35 75 0)
+    (property "NC Audit 2" "NC J_EXP1.2" (at 35 75 0)
+      (effects (font (size 1.27 1.27)) hide))
+    (property "NC Audit 3" "NC J_EXP1.3" (at 35 75 0)
+      (effects (font (size 1.27 1.27)) hide))
+    (property "NC Audit 4" "NC J_EXP1.4" (at 35 75 0)
       (effects (font (size 1.27 1.27)) hide))
     (pin "1")
@@
     (pin "MP")
     (instances (project "pocket_card_controller"
-      (path "/2e13cb0c-6647-4fc9-a0db-5ca9b27d688a" (reference "J_EXP") (unit 1))))
+      (path "/2e13cb0c-6647-4fc9-a0db-5ca9b27d688a" (reference "J_EXP1") (unit 1))))
   )
   (symbol (lib_id "PocketCard:JST2") (at 35 130 0) (unit 1)
     (exclude_from_sim no) (in_bom yes) (on_board yes) (dnp no)
-    (property "Reference" "J_BAT_IN" (at 26.11 124.92 0)
+    (property "Reference" "J_BAT_IN1" (at 26.11 124.92 0)
       (effects (font (size 1.27 1.27))))
     (property "Value" "WAFER-GH1.25-2PWB" (at 35 140.16 0)
@@
     (pin "MP")
     (instances (project "pocket_card_controller"
-      (path "/2e13cb0c-6647-4fc9-a0db-5ca9b27d688a" (reference "J_BAT_IN") (unit 1))))
+      (path "/2e13cb0c-6647-4fc9-a0db-5ca9b27d688a" (reference "J_BAT_IN1") (unit 1))))
   )
   (symbol (lib_id "PocketCard:JST2") (at 185 130 0) (unit 1)
     (exclude_from_sim no) (in_bom yes) (on_board yes) (dnp no)
-    (property "Reference" "J_BAT_OUT" (at 176.11 124.92 0)
+    (property "Reference" "J_BAT_OUT1" (at 176.11 124.92 0)
       (effects (font (size 1.27 1.27))))
     (property "Value" "WAFER-GH1.25-2PWB" (at 185 140.16 0)
@@
     (pin "MP")
     (instances (project "pocket_card_controller"
-      (path "/2e13cb0c-6647-4fc9-a0db-5ca9b27d688a" (reference "J_BAT_OUT") (unit 1))))
+      (path "/2e13cb0c-6647-4fc9-a0db-5ca9b27d688a" (reference "J_BAT_OUT1") (unit 1))))
   )
   (symbol (lib_id "PocketCard:Mount") (at 255 130 0) (unit 1)
