File: hardware/pocket_card/electronics/pocket_card_controller.kicad_pcb (KiCad board)
At the start: 2 copper layers, 80.5 x 37 mm, 17 parts, among them U1 SOIC-28W_7.5x17.9mm_P1.27mm

Commit message: feat: validate native Pocket Card KiCad project
Routing:
- net GND: track 245.7 -> 246.2 mm
Changed lines of the file:
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@@
 	(segment
 		(start 63.625 74.15)
+		(end 67.5 68)
+		(width 0.2)
+		(layer "B.Cu")
+		(net "GND")
+	)
+	(segment
+		(start 67.5 68)
 		(end 70.825 66.95)
 		(width 0.2)
