File: hardware/pocket_card/electronics/pocket_card_controller.kicad_pcb (KiCad board)
At the start: 2 copper layers, 80.5 x 37 mm, 17 parts, among them U1 SOIC-28W_7.5x17.9mm_P1.27mm

Commit message: fix: center Pocket Card serialization controller
Parts:
- moved U1 4.24 mm to (41.3, 69.0)
Routing:
- net GND: track 248.4 -> 0.00 mm, vias 8 -> 4
- net +3V3: track 35.4 -> 64.4 mm, vias 2 -> 1
- net SIG_MUTE: track 28.5 -> 46.3 mm, vias 2 -> 0
- net SIG_DOWN: track 43.8 -> 32.6 mm
- net SIG_UP: track 26.5 -> 21.2 mm
- net SIG_RESET: track 17.1 -> 21.2 mm
- net SIG_LEFT: track 43.9 -> 40.5 mm
- net INT: track 36.4 -> 33.1 mm
- net SIG_RIGHT: track 24.1 -> 21.3 mm
- net SIG_ACTION: track 32.9 -> 35.1 mm
- net SIG_MENU: track 23.2 -> 25.3 mm
- net SDA: track 42.0 -> 40.0 mm
- net SCL: track 34.7 -> 35.4 mm
- net SIG_UNDO: track 18.5 -> 17.8 mm
